File: Project K+.kicad_pcb (KiCad board)
At the start: 2 copper layers, 3.4 x 3 mm, 2 parts, among them U1 ProMicro, U2 Cherry_MX_RGB

Commit message: Add correct references and footprints to components
Parts:
- added C1: 100nF, Capacitor_SMD:C_0603_1608Metric, F.Cu at (320.4, -10.0)
- added C10: 100nF, Capacitor_SMD:C_0603_1608Metric, F.Cu at (324.5, -4.98)
- added C11: 100nF, Capacitor_SMD:C_0603_1608Metric, F.Cu at (328.5, -11.4)
- added C12: 100nF, Capacitor_SMD:C_0603_1608Metric, F.Cu at (328.5, -8.92)
- added C13: 100nF, Capacitor_SMD:C_0603_1608Metric, F.Cu at (297.9, -17.7)
- added C14: 100nF, Capacitor_SMD:C_0603_1608Metric, F.Cu at (298.1, 9.89)
- added C15: 100nF, Capacitor_SMD:C_0603_1608Metric, F.Cu at (320.4, -12.5)
- added C16: 100nF, Capacitor_SMD:C_0603_1608Metric, F.Cu at (275.6, 33.3)
- added C17: 100nF, Capacitor_SMD:C_0603_1608Metric, F.Cu at (324.3, -17.5)
- added C18: 100nF, Capacitor_SMD:C_0603_1608Metric, F.Cu at (320.4, -15.0)
- added C19: 100nF, Capacitor_SMD:C_0603_1608Metric, F.Cu at (306.1, 11.0)
- added C2: 100nF, Capacitor_SMD:C_0603_1608Metric, F.Cu at (302.1, 17.4)
- added C20: 100nF, Capacitor_SMD:C_0603_1608Metric, F.Cu at (306.1, 13.5)
- added C3: 100nF, Capacitor_SMD:C_0603_1608Metric, F.Cu at (320.4, -2.47)
- added C4: 100nF, Capacitor_SMD:C_0603_1608Metric, F.Cu at (316.0, 2.13)
- added C5: 100nF, Capacitor_SMD:C_0603_1608Metric, F.Cu at (298.9, 19.9)
- added C6: 100nF, Capacitor_SMD:C_0603_1608Metric, F.Cu at (290.0, 28.0)
- added C7: 100nF, Capacitor_SMD:C_0603_1608Metric, F.Cu at (314.6, 4.64)
- added C8: 100nF, Capacitor_SMD:C_0603_1608Metric, F.Cu at (275.6, 43.4)
- added C9: 100nF, Capacitor_SMD:C_0603_1608Metric, F.Cu at (283.6, 35.9)
- added D1: D_ALT, Diode_THT:D_DO-41_SOD81_P10.16mm_Horizontal, F.Cu at (295.0, -12.8)
- added D10: D_ALT, Diode_THT:D_DO-41_SOD81_P10.16mm_Horizontal, F.Cu at (311.7, -29.6)
- added D11: D_ALT, Diode_THT:D_DO-41_SOD81_P10.16mm_Horizontal, F.Cu at (239.2, 37.3)
- added D12: D_ALT, Diode_THT:D_DO-41_SOD81_P10.16mm_Horizontal, F.Cu at (297.8, -29.6)
- added D13: D_ALT, Diode_THT:D_DO-41_SOD81_P10.16mm_Horizontal, F.Cu at (281.1, -12.8)
- added D14: D_ALT, Diode_THT:D_DO-41_SOD81_P10.16mm_Horizontal, F.Cu at (225.3, 41.6)
- added D15: D_ALT, Diode_THT:D_DO-41_SOD81_P10.16mm_Horizontal, F.Cu at (211.4, 41.6)
- added D16: D_ALT, Diode_THT:D_DO-41_SOD81_P10.16mm_Horizontal, F.Cu at (225.3, 37.3)
- added D17: D_ALT, Diode_THT:D_DO-41_SOD81_P10.16mm_Horizontal, F.Cu at (197.5, 41.6)
- added D18: D_ALT, Diode_THT:D_DO-41_SOD81_P10.16mm_Horizontal, F.Cu at (211.4, 37.3)
- added D19: D_ALT, Diode_THT:D_DO-41_SOD81_P10.16mm_Horizontal, F.Cu at (264.3, 20.6)
- added D2: D_ALT, Diode_THT:D_DO-41_SOD81_P10.16mm_Horizontal, F.Cu at (253.1, 37.3)
- added D20: D_ALT, Diode_THT:D_DO-41_SOD81_P10.16mm_Horizontal, F.Cu at (281.1, -4.34)
- added D3: D_ALT, Diode_THT:D_DO-41_SOD81_P10.16mm_Horizontal, F.Cu at (281.1, -0.09)
- added D4: D_ALT, Diode_THT:D_DO-41_SOD81_P10.16mm_Horizontal, F.Cu at (281.1, -8.59)
- added D5: D_ALT, Diode_THT:D_DO-41_SOD81_P10.16mm_Horizontal, F.Cu at (297.8, -21.1)
- added D6: D_ALT, Diode_THT:D_DO-41_SOD81_P10.16mm_Horizontal, F.Cu at (197.5, 37.3)
- added D7: D_ALT, Diode_THT:D_DO-41_SOD81_P10.16mm_Horizontal, F.Cu at (297.8, -25.3)
- added D8: D_ALT, Diode_THT:D_DO-41_SOD81_P10.16mm_Horizontal, F.Cu at (239.2, 41.6)
- added D9: D_ALT, Diode_THT:D_DO-41_SOD81_P10.16mm_Horizontal, F.Cu at (281.1, 4.16)
- added J1: USB_C_Receptacle_USB2.0, Connector_USB:USB_C_Receptacle_HRO_TYPE-C-31-M-12, F.Cu at (383.2, -25.9)
- added J2: USB Breakout, Connector_PinHeader_2.54mm:PinHeader_1x04_P2.54mm_Vertical, F.Cu at (375.0, -29.4)
- added J3: RGB Breakout, Connector_PinHeader_2.54mm:PinHeader_1x03_P2.54mm_Vertical, F.Cu at (264.8, 25.1)
- added R1: 33R, Resistor_SMD:R_0603_1608Metric, F.Cu at (306.5, 5.95)
- added R10: 33R, Resistor_SMD:R_0603_1608Metric, F.Cu at (273.1, 30.4)
- added R11: 33R, Resistor_SMD:R_0603_1608Metric, F.Cu at (301.9, -17.7)
- added R12: 33R, Resistor_SMD:R_0603_1608Metric, F.Cu at (305.9, -17.7)
- added R13: 33R, Resistor_SMD:R_0603_1608Metric, F.Cu at (253.2, 40.7)
- added R14: 100R, Resistor_SMD:R_0603_1608Metric, F.Cu at (257.2, 40.7)
- added R15: 100R, Resistor_SMD:R_0603_1608Metric, F.Cu at (253.2, 43.2)
- added R16: 100R, Resistor_SMD:R_0603_1608Metric, F.Cu at (257.2, 43.2)
- added R17: 100R, Resistor_SMD:R_0603_1608Metric, F.Cu at (328.7, -21.5)
- added R18: 33R, Resistor_SMD:R_0603_1608Metric, F.Cu at (324.5, -15.0)
- added R19: 33R, Resistor_SMD:R_0603_1608Metric, F.Cu at (328.7, -24.0)
- added R2: 33R, Resistor_SMD:R_0603_1608Metric, F.Cu at (328.5, -16.4)
- added R20: 33R, Resistor_SMD:R_0603_1608Metric, F.Cu at (320.3, -17.5)
- added R21: 33R, Resistor_SMD:R_0603_1608Metric, F.Cu at (261.2, 40.7)
- added R22: 33R, Resistor_SMD:R_0603_1608Metric, F.Cu at (269.1, 30.4)
- added R23: 33R, Resistor_SMD:R_0603_1608Metric, F.Cu at (279.6, 35.9)
- added R24: 33R, Resistor_SMD:R_0603_1608Metric, F.Cu at (286.8, 20.4)
- added R25: 100R, Resistor_SMD:R_0603_1608Metric, F.Cu at (286.8, 22.9)
- added R26: 33R, Resistor_SMD:R_0603_1608Metric, F.Cu at (328.7, -19.0)
- added R27: 100R, Resistor_SMD:R_0603_1608Metric, F.Cu at (261.2, 43.2)
- added R28: 100R, Resistor_SMD:R_0603_1608Metric, F.Cu at (306.5, 3.44)
- added R29: 100R, Resistor_SMD:R_0603_1608Metric, F.Cu at (298.1, 12.4)
- added R3: 5.1K, Resistor_SMD:R_0603_1608Metric, F.Cu at (374.7, -18.2)
- added R30: 100R, Resistor_SMD:R_0603_1608Metric, F.Cu at (324.5, -12.5)
- added R31: 33R, Resistor_SMD:R_0603_1608Metric, F.Cu at (290.8, 20.4)
- added R32: 33R, Resistor_SMD:R_0603_1608Metric, F.Cu at (302.1, 9.89)
- added R33: 33R, Resistor_SMD:R_0603_1608Metric, F.Cu at (320.0, 0.04)
- added R34: 33R, Resistor_SMD:R_0603_1608Metric, F.Cu at (312.0, -0.38)
- added R35: 33R, Resistor_SMD:R_0603_1608Metric, F.Cu at (320.4, -7.49)
- added R36: 33R, Resistor_SMD:R_0603_1608Metric, F.Cu at (275.6, 35.9)
- added R37: 33R, Resistor_SMD:R_0603_1608Metric, F.Cu at (294.9, 20.4)
- added R38: 33R, Resistor_SMD:R_0603_1608Metric, F.Cu at (302.1, 12.4)
- added R39: 33R, Resistor_SMD:R_0603_1608Metric, F.Cu at (324.5, -10.0)
- added R4: 5.1K, Resistor_SMD:R_0603_1608Metric, F.Cu at (341.6, 0.07)
- added R40: 33R, Resistor_SMD:R_0603_1608Metric, F.Cu at (312.0, 2.13)
- added R41: 33R, Resistor_SMD:R_0603_1608Metric, F.Cu at (316.0, -0.38)
- added R42: 33R, Resistor_SMD:R_0603_1608Metric, F.Cu at (320.4, -4.98)
- added R43: 100R, Resistor_SMD:R_0603_1608Metric, F.Cu at (298.1, 17.4)
- added R44: 100R, Resistor_SMD:R_0603_1608Metric, F.Cu at (306.5, 8.46)
- added R45: 100R, Resistor_SMD:R_0603_1608Metric, F.Cu at (328.5, -13.9)
- added R46: 100R, Resistor_SMD:R_0603_1608Metric, F.Cu at (290.8, 22.9)
- added R47: 100R, Resistor_SMD:R_0603_1608Metric, F.Cu at (324.5, -7.49)
- added R48: 33R, Resistor_SMD:R_0603_1608Metric, F.Cu at (298.9, 22.4)
- added R49: 33R, Resistor_SMD:R_0603_1608Metric, F.Cu at (283.6, 38.4)
- added R5: 220R, Resistor_SMD:R_0603_1608Metric, F.Cu at (337.6, 0.07)
- added R50: 33R, Resistor_SMD:R_0603_1608Metric, F.Cu at (287.6, 33.0)
- added R51: 33R, Resistor_SMD:R_0603_1608Metric, F.Cu at (279.6, 40.9)
- added R52: 33R, Resistor_SMD:R_0603_1608Metric, F.Cu at (310.6, 9.66)
- added R53: 33R, Resistor_SMD:R_0603_1608Metric, F.Cu at (294.9, 25.5)
- added R54: 33R, Resistor_SMD:R_0603_1608Metric, F.Cu at (290.0, 30.5)
- added R55: 33R, Resistor_SMD:R_0603_1608Metric, F.Cu at (294.9, 22.9)
- added R56: 33R, Resistor_SMD:R_0603_1608Metric, F.Cu at (286.0, 28.0)
- added R57: 33R, Resistor_SMD:R_0603_1608Metric, F.Cu at (290.8, 25.5)
- added R58: 100R, Resistor_SMD:R_0603_1608Metric, F.Cu at (310.6, 4.64)
- added R59: 100R, Resistor_SMD:R_0603_1608Metric, F.Cu at (286.0, 30.5)
- added R6: 33R, Resistor_SMD:R_0603_1608Metric, F.Cu at (286.8, 25.5)
- added R60: 100R, Resistor_SMD:R_0603_1608Metric, F.Cu at (275.6, 40.9)
- added R61: 100R, Resistor_SMD:R_0603_1608Metric, F.Cu at (283.6, 33.3)
- added R62: 100R, Resistor_SMD:R_0603_1608Metric, F.Cu at (302.1, 14.9)
- added R63: 100R, Resistor_SMD:R_0603_1608Metric, F.Cu at (279.6, 38.4)
- added R64: 33R, Resistor_SMD:R_0603_1608Metric, F.Cu at (310.6, 7.15)
- added R7: 33R, Resistor_SMD:R_0603_1608Metric, F.Cu at (279.6, 33.3)
- added R8: 33R, Resistor_SMD:R_0603_1608Metric, F.Cu at (275.6, 38.4)
- added R9: 33R, Resistor_SMD:R_0603_1608Metric, F.Cu at (298.1, 14.9)
- added SW1: Rotary_Encoder_Switch, Rotary_Encoder:RotaryEncoder_Alps_EC11E-Switch_Vertical_H20mm, F.Cu at (337.6, -26.6)
- added SW2: Rotary_Encoder_Switch, Rotary_Encoder:RotaryEncoder_Alps_EC11E-Switch_Vertical_H20mm, F.Cu at (337.6, -11.3)
- added SW3: Rotary_Encoder_Switch, Rotary_Encoder:RotaryEncoder_Alps_EC11E-Switch_Vertical_H20mm, F.Cu at (356.1, -26.6)
- added SW4: Rotary_Encoder_Switch, Rotary_Encoder:RotaryEncoder_Alps_EC11E-Switch_Vertical_H20mm, F.Cu at (356.1, -11.3)
- added U10: Cherry_MX_RGB, Cherry_MX_SMD:Cherry-MX_PCB-Mounted_LTST-A683CEGBW_Mill-Max-7305, F.Cu at (223.8, -26.2)
- added U11: WS2811, Package_SO:SOP-8_3.9x4.9mm_P1.27mm, F.Cu at (297.3, -7.49)
- added U12: WS2811, Package_SO:SOP-8_3.9x4.9mm_P1.27mm, F.Cu at (314.0, -24.2)
- added U13: WS2811, Package_SO:SOP-8_3.9x4.9mm_P1.27mm, F.Cu at (280.6, 22.4)
- added U14: Cherry_MX_RGB, Cherry_MX_SMD:Cherry-MX_PCB-Mounted_LTST-A683CEGBW_Mill-Max-7305, F.Cu at (220.7, -6.61)
- added U15: WS2811, Package_SO:SOP-8_3.9x4.9mm_P1.27mm, F.Cu at (327.9, -28.5)
- added U16: Cherry_MX_RGB, Cherry_MX_SMD:Cherry-MX_PCB-Mounted_LTST-A683CEGBW_Mill-Max-7305, F.Cu at (203.9, 10.1)
- added U17: Cherry_MX_RGB, Cherry_MX_SMD:Cherry-MX_PCB-Mounted_LTST-A683CEGBW_Mill-Max-7305, F.Cu at (223.8, -45.2)
- added U18: Cherry_MX_RGB, Cherry_MX_SMD:Cherry-MX_PCB-Mounted_LTST-A683CEGBW_Mill-Max-7305, F.Cu at (220.7, 26.8)
- added U19: Cherry_MX_RGB, Cherry_MX_SMD:Cherry-MX_PCB-Mounted_LTST-A683CEGBW_Mill-Max-7305, F.Cu at (203.9, -6.61)
- added U2: WS2811, Package_SO:SOP-8_3.9x4.9mm_P1.27mm, F.Cu at (271.3, 25.9)
- added U20: WS2811, Package_SO:SOP-8_3.9x4.9mm_P1.27mm, F.Cu at (283.4, 9.51)
- added U21: WS2811, Package_SO:SOP-8_3.9x4.9mm_P1.27mm, F.Cu at (283.4, 16.0)
- added U22: WS2811, Package_SO:SOP-8_3.9x4.9mm_P1.27mm, F.Cu at (314.2, -4.86)
- added U23: WS2811, Package_SO:SOP-8_3.9x4.9mm_P1.27mm, F.Cu at (314.2, -11.3)
- added U24: WS2811, Package_SO:SOP-8_3.9x4.9mm_P1.27mm, F.Cu at (322.5, -22.0)
- added U25: Cherry_MX_RGB, Cherry_MX_SMD:Cherry-MX_PCB-Mounted_LTST-A683CEGBW_Mill-Max-7305, F.Cu at (203.9, 26.8)
- added U26: WS2811, Package_SO:SOP-8_3.9x4.9mm_P1.27mm, F.Cu at (291.9, 16.0)
- added U27: Cherry_MX_RGB, Cherry_MX_SMD:Cherry-MX_PCB-Mounted_LTST-A683CEGBW_Mill-Max-7305, F.Cu at (237.4, -6.61)
- added U28: Cherry_MX_RGB, Cherry_MX_SMD:Cherry-MX_PCB-Mounted_LTST-A683CEGBW_Mill-Max-7305, F.Cu at (254.1, -23.3)
- added U29: Cherry_MX_RGB, Cherry_MX_SMD:Cherry-MX_PCB-Mounted_LTST-A683CEGBW_Mill-Max-7305, F.Cu at (204.8, -26.2)
- added U3: WS2811, Package_SO:SOP-8_3.9x4.9mm_P1.27mm, F.Cu at (269.4, 35.6)
- added U30: Cherry_MX_RGB, Cherry_MX_SMD:Cherry-MX_PCB-Mounted_LTST-A683CEGBW_Mill-Max-7305, F.Cu at (237.4, 10.1)
- added U31: WS2811, Package_SO:SOP-8_3.9x4.9mm_P1.27mm, F.Cu at (300.3, 5.41)
- added U32: WS2811, Package_SO:SOP-8_3.9x4.9mm_P1.27mm, F.Cu at (305.8, -1.04)
- added U33: WS2811, Package_SO:SOP-8_3.9x4.9mm_P1.27mm, F.Cu at (279.8, 28.9)
- added U34: WS2811, Package_SO:SOP-8_3.9x4.9mm_P1.27mm, F.Cu at (269.4, 42.1)
- added U35: WS2811, Package_SO:SOP-8_3.9x4.9mm_P1.27mm, F.Cu at (291.9, 9.51)
- added U36: Cherry_MX_RGB, Cherry_MX_SMD:Cherry-MX_PCB-Mounted_LTST-A683CEGBW_Mill-Max-7305, F.Cu at (237.4, 26.8)
- added U37: Cherry_MX_RGB, Cherry_MX_SMD:Cherry-MX_PCB-Mounted_LTST-A683CEGBW_Mill-Max-7305, F.Cu at (254.1, 10.1)
- added U38: Cherry_MX_RGB, Cherry_MX_SMD:Cherry-MX_PCB-Mounted_LTST-A683CEGBW_Mill-Max-7305, F.Cu at (270.8, -6.61)
- added U39: Cherry_MX_RGB, Cherry_MX_SMD:Cherry-MX_PCB-Mounted_LTST-A683CEGBW_Mill-Max-7305, F.Cu at (287.5, -23.3)
- added U4: WS2811, Package_SO:SOP-8_3.9x4.9mm_P1.27mm, F.Cu at (297.3, -1.04)
- added U40: Cherry_MX_RGB, Cherry_MX_SMD:Cherry-MX_PCB-Mounted_LTST-A683CEGBW_Mill-Max-7305, F.Cu at (254.1, 26.8)
- added U41: Cherry_MX_RGB, Cherry_MX_SMD:Cherry-MX_PCB-Mounted_LTST-A683CEGBW_Mill-Max-7305, F.Cu at (270.8, 10.1)
- added U5: WS2811, Package_SO:SOP-8_3.9x4.9mm_P1.27mm, F.Cu at (305.8, -7.49)
- added U6: WS2811, Package_SO:SOP-8_3.9x4.9mm_P1.27mm, F.Cu at (314.0, -17.8)
- added U7: Cherry_MX_RGB, Cherry_MX_SMD:Cherry-MX_PCB-Mounted_LTST-A683CEGBW_Mill-Max-7305, F.Cu at (270.8, -23.3)
- added U8: Cherry_MX_RGB, Cherry_MX_SMD:Cherry-MX_PCB-Mounted_LTST-A683CEGBW_Mill-Max-7305, F.Cu at (254.1, -6.61)
- added U9: Cherry_MX_RGB, Cherry_MX_SMD:Cherry-MX_PCB-Mounted_LTST-A683CEGBW_Mill-Max-7305, F.Cu at (220.7, 10.1)
- moved U2 136.0 mm to (204.8, -45.2)
- turned U1 to 270 degrees
Connections:
- U1 pad 10: Net-(U1-Pad10) -> Col2
- U1 pad 11: Net-(U1-Pad11) -> Col1
- U1 pad 12: Net-(U1-Pad12) -> Col0
- U1 pad 13: Net-(U1-Pad13) -> RGB
- U1 pad 2: Net-(U1-Pad2) -> Row4
- U1 pad 21: Net-(U1-Pad21) -> +5V
- U1 pad 23: Net-(U1-Pad23) -> GND
- U1 pad 3: Net-(U1-Pad3) -> GND
- U1 pad 4: Net-(U1-Pad4) -> GND
- U1 pad 5: Net-(U1-Pad5) -> Row3
- U1 pad 6: Net-(U1-Pad6) -> Row2
- U1 pad 7: Net-(U1-Pad7) -> Row1
- U1 pad 8: Net-(U1-Pad8) -> Row0
- U1 pad 9: Net-(U1-Pad9) -> Col3

Commit message: Commit
Parts:
- removed the U2 at (204.8, -45.2)
- C1, C20, C6: value 100nF -> C
- C10: renamed from C7; value 100nF -> C
- C11: renamed from C12; value 100nF -> C
- C12: renamed from C18; value 100nF -> C
- C13: renamed from C4; value 100nF -> C
- C14: renamed from C8; value 100nF -> C
- C15: renamed from C14; value 100nF -> C
- C16: renamed from C19; value 100nF -> C
- C17: renamed from C5; value 100nF -> C
- C18: renamed from C9; value 100nF -> C
- C19: renamed from C15; value 100nF -> C
- C2: renamed from C13; value 100nF -> C
- C3: renamed from C10; value 100nF -> C
- C4: renamed from C16; value 100nF -> C
- C5: renamed from C2; value 100nF -> C
- C7: renamed from C11; value 100nF -> C
- C8: renamed from C17; value 100nF -> C
- C9: renamed from C3; value 100nF -> C
- D1, D20, D6, J1, J2, U1, U2: moved to B.Cu
- D10: renamed from D7; moved to B.Cu
- D11: renamed from D12; moved to B.Cu
- D12: renamed from D18; moved to B.Cu
- D13: renamed from D4; moved to B.Cu
- D14: renamed from D8; moved to B.Cu
- D15: renamed from D14; moved to B.Cu
- D16: renamed from D19; moved to B.Cu
- D17: renamed from D5; moved to B.Cu
- D18: renamed from D9; moved to B.Cu
- D19: renamed from D15; moved to B.Cu
- D2: renamed from D13; moved to B.Cu
- D3: renamed from D10; moved to B.Cu
- D4: renamed from D16; moved to B.Cu
- D5: renamed from D2; moved to B.Cu
- D7: renamed from D11; moved to B.Cu
- D8: renamed from D17; moved to B.Cu
- D9: renamed from D3; moved to B.Cu
- J3: value RGB Breakout -> Conn_01x03_Male; footprint Connector_PinHeader_2.54mm:PinHeader_1x03_P2.54mm_Vertical -> Connector_PinHeader_2.54mm:PinHeader_1x03_P2.54mm_Horizontal
- R10: renamed from R31; value 33R -> R
- R11: renamed from R48; value 33R -> R
- R12: renamed from R2; value 33R -> R
- R13: renamed from R38; value 33R -> R
- R14: renamed from R32; value 33R -> R
- R15: renamed from R49; value 33R -> R
- R16: renamed from R14; value 100R -> R
- R17: renamed from R27; value 100R -> R
- R18: renamed from R44; value 100R -> R
- R19: renamed from R59; value 100R -> R
- R20: renamed from R6; value 33R -> R
- R21: renamed from R18; value 33R -> R
- R22: renamed from R33; value 33R -> R
- R23: renamed from R50; value 33R -> R
- R24: renamed from R7; value 33R -> R
- R25: renamed from R19; value 33R -> R
- R26: renamed from R34; value 33R -> R
- R27: renamed from R51; value 33R -> R
- R28: renamed from R15; value 100R -> R
- R29: renamed from R28; value 100R -> R
- R30: renamed from R45; value 100R -> R
- R31: renamed from R60; value 100R -> R
- R32: renamed from R8; value 33R -> R
- R33: renamed from R20; value 33R -> R
- R34: renamed from R35; value 33R -> R
- R35: renamed from R52; value 33R -> R
- R36: renamed from R9; value 33R -> R
- R37: renamed from R21; value 33R -> R
- R38: renamed from R36; value 33R -> R
- R39: renamed from R53; value 33R -> R
- R4: renamed from R25; value 100R -> R
- R40: renamed from R16; value 100R -> R
- R41: renamed from R29; value 100R -> R
- R42: renamed from R46; value 100R -> R
- R43: renamed from R62; value 100R -> R
- R44: renamed from R10; value 33R -> R
- R45: renamed from R22; value 33R -> R
- R46: renamed from R39; value 33R -> R
- R47: renamed from R54; value 33R -> R
- R48: renamed from R11; value 33R -> R
- R49: renamed from R23; value 33R -> R
- R5: renamed from R61; value 100R -> R
- R50: renamed from R40; value 33R -> R
- R51: renamed from R55; value 33R -> R
- R52: renamed from R17; value 100R -> R
- R53: renamed from R30; value 100R -> R
- R54: renamed from R47; value 100R -> R
- R55: renamed from R63; value 100R -> R
- R56: renamed from R12; value 33R -> R
- R57: renamed from R24; value 33R -> R
- R58: renamed from R41; value 33R -> R
- R59: renamed from R56; value 33R -> R
- R6: renamed from R43; value 100R -> R
- R60: renamed from R13; value 33R -> R
- R61: renamed from R26; value 33R -> R
- R62: renamed from R42; value 33R -> R
- R63: renamed from R57; value 33R -> R
- R64: value 33R -> R
- R7: renamed from R58; value 100R -> R
- R8: renamed from R1; value 33R -> R
- R9: renamed from R37; value 33R -> R
- U10: renamed from U4; moved to B.Cu
- U11: renamed from U12; moved to B.Cu
- U12: renamed from U22; moved to B.Cu
- U13: renamed from U33; moved to B.Cu
- U14: renamed from U5; moved to B.Cu
- U15: renamed from U13; moved to B.Cu
- U16: renamed from U23; moved to B.Cu
- U17: renamed from U34; moved to B.Cu
- U18: renamed from U6; moved to B.Cu
- U19: renamed from U15; moved to B.Cu
- U20: renamed from U24; moved to B.Cu
- U21: renamed from U35; moved to B.Cu
- U3: renamed from U26; moved to B.Cu
- U4: renamed from U20; moved to B.Cu
- U5: renamed from U31; moved to B.Cu
- U6: renamed from U3; moved to B.Cu
- U7: renamed from U11; moved to B.Cu
- U8: renamed from U21; moved to B.Cu
- U9: renamed from U32; moved to B.Cu
- moved J1 293.6 mm to (95.2, 31.6)
- moved J2 293.3 mm to (91.4, 45.4), turned to 270 degrees
- moved SW1 256.4 mm to (95.2, 57.1), turned to 90 degrees
- moved SW3 238.0 mm to (133.3, 57.1), turned to 90 degrees
- moved SW2 233.6 mm to (114.3, 57.1), turned to 90 degrees
- moved MX17 220.1 mm to (95.2, 152.4)
- moved SW4 214.9 mm to (152.4, 57.1), turned to 90 degrees
- moved D1 212.2 mm to (104.8, 81.3), turned to 90 degrees
- moved MX5 211.9 mm to (95.2, 95.2)
- moved D3 202.0 mm to (142.9, 81.3), turned to 90 degrees
- moved MX9 199.6 mm to (95.2, 114.3)
- moved MX10 193.5 mm to (114.3, 114.3)
- moved MX12 192.9 mm to (152.4, 114.3)
- moved MX20 185.1 mm to (152.4, 152.4)
- moved D2 183.3 mm to (123.8, 81.3), turned to 90 degrees
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- renumbered U14 to MX1, U17 to MX10, U28 to MX11, U39 to MX12, U9 to MX13, U18 to MX14, U29 to MX15, U40 to MX16, U10 to MX17, U19 to MX18, U30 to MX19, U38 to MX2, U41 to MX20, U25 to MX3, U36 to MX4, U7 to MX5, U16 to MX6, U27 to MX7, U37 to MX8, U8 to MX9, R3 to R1, R4 to R2, R5 to R3
Other:
- board size 3.4 x 3 mm -> 76.2 x 133.4 mm

Commit message: commit
Parts:
- added R65: 220R, Resistor_SMD:R_0603_1608Metric, B.Cu at (103.6, 50.0)
- added R66: 220R, Resistor_SMD:R_0603_1608Metric, B.Cu at (122.6, 50.0)
- added R67: 220R, Resistor_SMD:R_0603_1608Metric, B.Cu at (141.7, 50.0)
- C1, C10, C11, C12, C13, C14, C15, C16, C17, C18, C19, C2, C20, C3, C4, C5, C6, C7, C8, C9: value C -> 100n; moved to B.Cu
- D1, D11, D13, D15, D17, D19, D3, D5, D7, D9: footprint Diode_THT:D_DO-41_SOD81_P10.16mm_Horizontal -> Diode_SMD:D_SOD-123F
- D10, D12, D14, D16, D18, D2, D20, D4, D6, D8: footprint Diode_THT:D_DO-41_SOD81_P10.16mm_Horizontal -> Diode_SMD:D_SOD-123F; moved to F.Cu
- R1, R2, R3: moved to B.Cu
- R10, R11, R12, R13, R14, R15, R20, R21, R22, R23, R24, R25, R26, R27, R32, R33, R34, R35, R36, R37, R38, R39, R44, R45, R46, R47, R48, R49, R50, R51, R56, R57, R58, R59, R60, R61, R62, R63, R64, R8, R9: value R -> 33R
- R16, R17, R18, R19, R28, R29, R30, R31, R4, R40, R41, R42, R43, R5, R52, R53, R54, R55, R6, R7: value R -> 100R
- moved R1 288.3 mm to (92.9, 42.9)
- moved C19 257.2 mm to (123.8, 153.3)
- moved C13 253.8 mm to (104.8, 142.9)
- moved C9 249.9 mm to (104.8, 123.8)
- moved R2 247.7 mm to (97.6, 42.9)
- moved C11 243.9 mm to (123.8, 123.8)
- moved C1 236.0 mm to (104.8, 85.7)
- moved C7 235.3 mm to (123.8, 104.8)
- moved C17 235.0 mm to (104.8, 152.4)
- moved C12 225.4 mm to (142.9, 123.8)
- moved C3 220.2 mm to (123.8, 85.7)
- moved C10 220.0 mm to (123.8, 114.3)
- moved C15 219.2 mm to (123.8, 142.9)
- moved C8 218.8 mm to (142.9, 104.8)
- moved C5 215.8 mm to (104.8, 104.8)
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Connections:
- SW1 pad S2: Net-(SW1-PadS2) -> GND
- SW2 pad S2: Net-(SW2-PadS2) -> GND
- SW3 pad S2: Net-(SW3-PadS2) -> GND
- U1 pad 14: Net-(U1-Pad14) -> SW1
- U1 pad 15: Net-(U1-Pad15) -> SW2
- U1 pad 16: Net-(U1-Pad16) -> SW3
- U1 pad 17: Net-(U1-Pad17) -> SW4
Routing:
- net Row4: track 0.00 -> 141.4 mm
- net Row3: track 0.00 -> 127.6 mm
- net Row2: track 0.00 -> 124.4 mm
- net Col0: track 0.00 -> 99.1 mm
- net Row1: track 0.00 -> 96.3 mm
- net Col1: track 0.00 -> 85.9 mm
- net +5V: track 0.00 -> 74.1 mm, vias 0 -> 1
- net Row0: track 0.00 -> 63.6 mm
- net Col3: track 0.00 -> 62.1 mm
- net GND: track 0.00 -> 61.6 mm, vias 0 -> 1
- net Col2: track 0.00 -> 47.1 mm
- net SW4: track 0.00 -> 47.0 mm
- net SW3: track 0.00 -> 29.9 mm
- net SW2: track 0.00 -> 15.8 mm
- net Net-(D18-Pad2): track 0.00 -> 14.2 mm
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