File: Project K+.kicad_pcb (KiCad board)
At the start: 2 copper layers, 271 parts, among them J1 USB_C_Receptacle_USB2.0, J2 USB Breakout, SW10 F5, SW100 LSPACE, SW101 RSPACE, SW102 ALTGR, SW103 FN, SW104 MENU, SW105 RCTRL, SW106 LEFT, SW107 DOWN, SW108 RIGHT, SW109 MACRO17, SW11 F6, SW110 MACRO18, SW111 MACRO19, SW112 MACRO20, SW12 F7, SW13 F8, SW14 F9, SW15 F10, SW16 F11, SW17 F12, SW18 PRTSCR, SW19 SCRLOCK, SW20 PAUSE, SW21 `, SW22 1, SW23 2, SW24 3, SW25 4, SW26 5, SW27 6, SW28 7, SW29 8, SW30 9, SW31 0, SW32 -, SW33 =, SW34 BACKSPACE, SW35 INSERT, SW36 HOME, SW37 PGUP, SW38 MACRO1, SW39 MACRO2, SW40 MACRO3, SW41 MACRO4, SW42 TAB, SW43 Q, SW44 W, SW45 E, SW46 R, SW47 T, SW48 Y, SW49 U, SW5 ESC, SW50 I, SW51 O, SW52 P, SW53 [, SW54 ], SW55 \, SW56 DEL, SW57 END, SW58 PGDN, SW59 MACRO5, SW6 F1, SW60 MACRO6, SW61 MACRO7, SW62 MACRO8, SW63 CAPSLOCK, SW64 A, SW65 S, SW66 D, SW67 F, SW68 G, SW69 H, SW7 F2, SW70 J, SW71 K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

Commit message: Add USB ports
Parts:
- removed ARD1: ProMicro, Arduino_Pro_Micro:ProMicro
- removed J2: USB Breakout, Connector_PinHeader_2.54mm:PinHeader_1x04_P2.54mm_Vertical
- added 7SD1: SA39-11EWA, Display_7Segment:Sx39-1xxxxx, F.Cu at (313.5, 193.4)
- added 7SD2: SA39-11EWA, Display_7Segment:Sx39-1xxxxx, F.Cu at (351.6, 193.4)
- added C1: 1uF, Capacitor_SMD:C_0603_1608Metric, F.Cu at (114.6, -13.7)
- added C10: 20pF, Capacitor_SMD:C_0603_1608Metric, F.Cu at (137.1, 16.1)
- added C11: 20pF, Capacitor_SMD:C_0603_1608Metric, F.Cu at (129.0, 16.1)
- added C12: 0.1uF, Capacitor_SMD:C_0603_1608Metric, F.Cu at (133.0, 16.1)
- added C13: 0.1uF, Capacitor_SMD:C_0603_1608Metric, F.Cu at (137.1, 13.5)
- added C14: 1uF, Capacitor_SMD:C_0603_1608Metric, F.Cu at (133.0, 13.5)
- added C15: 1uF, Capacitor_SMD:C_0603_1608Metric, F.Cu at (125.0, 16.1)
- added C17: 1uF, Capacitor_SMD:C_0603_1608Metric, F.Cu at (125.0, 18.6)
- added C2: 20pF, Capacitor_SMD:C_0603_1608Metric, F.Cu at (119.1, -17.8)
- added C20: 20pF, Capacitor_SMD:C_0603_1608Metric, F.Cu at (176.4, -2.81)
- added C21: 20pF, Capacitor_SMD:C_0603_1608Metric, F.Cu at (165.1, 8.09)
- added C23: 0.1uF, Capacitor_SMD:C_0603_1608Metric, F.Cu at (172.4, -0.30)
- added C25: 1uF, Capacitor_SMD:C_0603_1608Metric, F.Cu at (125.0, 13.5)
- added C3: 20pF, Capacitor_SMD:C_0603_1608Metric, F.Cu at (114.6, -11.2)
- added C4: 0.1uF, Capacitor_SMD:C_0603_1608Metric, F.Cu at (118.6, -13.7)
- added C5: 1uF, Capacitor_SMD:C_0603_1608Metric, F.Cu at (123.1, -17.8)
- added C6: 1uF, Capacitor_SMD:C_0603_1608Metric, F.Cu at (141.1, 13.5)
- added C7: 1uF, Capacitor_SMD:C_0603_1608Metric, F.Cu at (129.0, 18.6)
- added C8: 20pF, Capacitor_SMD:C_0603_1608Metric, F.Cu at (133.0, 18.6)
- added C9: 20pF, Capacitor_SMD:C_0603_1608Metric, F.Cu at (149.0, 5.58)
- added D1: LED, Capacitor_SMD:C_0603_1608Metric, F.Cu at (114.6, -8.71)
- added D11: LED, Capacitor_SMD:C_0603_1608Metric, F.Cu at (172.4, -12.8)
- added D14: G, Capacitor_SMD:C_0603_1608Metric, F.Cu at (141.1, 18.6)
- added D15: Y, Capacitor_SMD:C_0603_1608Metric, F.Cu at (149.0, 10.6)
- added D2: G, Capacitor_SMD:C_0603_1608Metric, F.Cu at (118.6, -11.2)
- added D3: Y, Capacitor_SMD:C_0603_1608Metric, F.Cu at (122.6, -15.3)
- added D4: LED, Capacitor_SMD:C_0603_1608Metric, F.Cu at (172.4, -15.4)
- added D5: LED, Capacitor_SMD:C_0603_1608Metric, F.Cu at (137.1, 18.6)
- added D6: G, Capacitor_SMD:C_0603_1608Metric, F.Cu at (168.4, -12.8)
- added D7: Y, Capacitor_SMD:C_0603_1608Metric, F.Cu at (145.0, 8.09)
- added D8: G, Capacitor_SMD:C_0603_1608Metric, F.Cu at (168.4, -10.3)
- added D9: Y, Capacitor_SMD:C_0603_1608Metric, F.Cu at (149.0, 8.09)
- added M3_SCREW_1: MountingHole, MountingHole:MountingHole_3.2mm_M3_Pad_Via, F.Cu at (2.70, 132.7)
- added M3_SCREW_10: MountingHole, MountingHole:MountingHole_3.2mm_M3_Pad_Via, F.Cu at (268.2, 218.4)
- added M3_SCREW_11: MountingHole, MountingHole:MountingHole_3.2mm_M3_Pad_Via, F.Cu at (326.5, 132.7)
- added M3_SCREW_12: MountingHole, MountingHole:MountingHole_3.2mm_M3_Pad_Via, F.Cu at (211.1, 172.0)
- added M3_SCREW_13: MountingHole, MountingHole:MountingHole_3.2mm_M3_Pad_Via, F.Cu at (345.6, 170.8)
- added M3_SCREW_14: MountingHole, MountingHole:MountingHole_3.2mm_M3_Pad_Via, F.Cu at (440.8, 208.9)
- added M3_SCREW_15: MountingHole, MountingHole:MountingHole_3.2mm_M3_Pad_Via, F.Cu at (326.5, 208.9)
- added M3_SCREW_16: MountingHole, MountingHole:MountingHole_3.2mm_M3_Pad_Via, F.Cu at (402.7, 208.9)
- added M3_SCREW_17: MountingHole, MountingHole:MountingHole_3.2mm_M3_Pad_Via, F.Cu at (402.7, 132.7)
- added M3_SCREW_18: MountingHole, MountingHole:MountingHole_3.2mm_M3_Pad_Via, F.Cu at (440.8, 132.7)
- added M3_SCREW_19: MountingHole, MountingHole:MountingHole_3.2mm_M3_Pad_Via, F.Cu at (421.8, 170.8)
- added M3_SCREW_2: MountingHole, MountingHole:MountingHole_3.2mm_M3_Pad_Via, F.Cu at (97.9, 132.7)
- added M3_SCREW_3: MountingHole, MountingHole:MountingHole_3.2mm_M3_Pad_Via, F.Cu at (158.7, 132.7)
- added M3_SCREW_4: MountingHole, MountingHole:MountingHole_3.2mm_M3_Pad_Via, F.Cu at (13.4, 180.3)
- added M3_SCREW_5: MountingHole, MountingHole:MountingHole_3.2mm_M3_Pad_Via, F.Cu at (93.2, 172.0)
- added M3_SCREW_6: MountingHole, MountingHole:MountingHole_3.2mm_M3_Pad_Via, F.Cu at (7.46, 218.4)
- added M3_SCREW_7: MountingHole, MountingHole:MountingHole_3.2mm_M3_Pad_Via, F.Cu at (253.9, 132.7)
- added M3_SCREW_8: MountingHole, MountingHole:MountingHole_3.2mm_M3_Pad_Via, F.Cu at (103.9, 218.4)
- added M3_SCREW_9: MountingHole, MountingHole:MountingHole_3.2mm_M3_Pad_Via, F.Cu at (144.4, 218.4)
- added R24: 1K, Resistor_SMD:R_0603_1608Metric, F.Cu at (114.6, -6.20)
- added R25: 10K, Resistor_SMD:R_0603_1608Metric, F.Cu at (118.6, -8.71)
- added R26: 22R, Resistor_SMD:R_0603_1608Metric, F.Cu at (122.6, -12.8)
- added R27: 22R, Resistor_SMD:R_0603_1608Metric, F.Cu at (118.6, -6.20)
- added R28: 330R, Resistor_SMD:R_0603_1608Metric, F.Cu at (122.6, -10.2)
- added R29: 330R, Resistor_SMD:R_0603_1608Metric, F.Cu at (122.6, -7.74)
- added R30: 1K, Resistor_SMD:R_0603_1608Metric, F.Cu at (168.4, -7.83)
- added R31: 1K, Resistor_SMD:R_0603_1608Metric, F.Cu at (145.1, 13.1)
- added R32: 10K, Resistor_SMD:R_0603_1608Metric, F.Cu at (153.0, 5.58)
- added R33: 10K, Resistor_SMD:R_0603_1608Metric, F.Cu at (172.4, -10.3)
- added R34: 5.1K, Resistor_SMD:R_0603_1608Metric, F.Cu at (153.0, 8.09)
- added R35: 5.1K, Resistor_SMD:R_0603_1608Metric, F.Cu at (141.1, 16.1)
- added R36: 5.1K, Resistor_SMD:R_0603_1608Metric, F.Cu at (176.4, -7.83)
- added R37: 5.1K, Resistor_SMD:R_0603_1608Metric, F.Cu at (168.4, -0.30)
- added R38: 22R, Resistor_SMD:R_0603_1608Metric, F.Cu at (157.1, 10.6)
- added R39: 22R, Resistor_SMD:R_0603_1608Metric, F.Cu at (145.1, 15.6)
- added R40: 22R, Resistor_SMD:R_0603_1608Metric, F.Cu at (161.1, 5.58)
- added R41: 22R, Resistor_SMD:R_0603_1608Metric, F.Cu at (153.1, 13.1)
- added R42: 330R, Resistor_SMD:R_0603_1608Metric, F.Cu at (149.1, 18.1)
- added R43: 330R, Resistor_SMD:R_0603_1608Metric, F.Cu at (172.4, -5.32)
- added R44: 330R, Resistor_SMD:R_0603_1608Metric, F.Cu at (157.1, 8.09)
- added R45: 330R, Resistor_SMD:R_0603_1608Metric, F.Cu at (153.1, 18.1)
- added R47: 1K, Resistor_SMD:R_0603_1608Metric, F.Cu at (172.4, -7.83)
- added R49: 10K, Resistor_SMD:R_0603_1608Metric, F.Cu at (149.1, 15.6)
- added R51: 5.1K, Resistor_SMD:R_0603_1608Metric, F.Cu at (149.1, 13.1)
- added R53: 5.1K, Resistor_SMD:R_0603_1608Metric, F.Cu at (145.1, 18.1)
- added R55: 22R, Resistor_SMD:R_0603_1608Metric, F.Cu at (168.4, -2.81)
- added R57: 22R, Resistor_SMD:R_0603_1608Metric, F.Cu at (165.1, 5.58)
- added R60: 330R, Resistor_SMD:R_0603_1608Metric, F.Cu at (172.4, -2.81)
- added R61: 330R, Resistor_SMD:R_0603_1608Metric, F.Cu at (161.1, 8.09)
- added U1: ATmega32U4-AU, Package_QFP:TQFP-44_10x10mm_P0.8mm, F.Cu at (105.4, -11.8)
- added U2: ATmega32U4-AU, Package_QFP:TQFP-44_10x10mm_P0.8mm, F.Cu at (135.8, 5.06)
- added U3: ATmega32U4-AU, Package_QFP:TQFP-44_10x10mm_P0.8mm, F.Cu at (135.8, -9.39)
- added U5: ATmega32U4-AU, Package_QFP:TQFP-44_10x10mm_P0.8mm, F.Cu at (121.3, 5.06)
- added USB3: USB_C_Receptacle_USB2.0, Connector_USB:USB_C_Receptacle_HRO_TYPE-C-31-M-12, B.Cu at (72.9, 101.8)
- added USB4: USB_C_Receptacle_USB2.0, Connector_USB:USB_C_Receptacle_HRO_TYPE-C-31-M-12, B.Cu at (87.2, 101.8)
- added USB5: USB_C_Receptacle_USB2.0, Connector_USB:USB_C_Receptacle_HRO_TYPE-C-31-M-12, B.Cu at (101.5, 101.8)
- added USB7: USB_C_Receptacle_USB2.0, Connector_USB:USB_C_Receptacle_HRO_TYPE-C-31-M-12, B.Cu at (336.1, 101.8)
- added USB8: USB_C_Receptacle_USB2.0, Connector_USB:USB_C_Receptacle_HRO_TYPE-C-31-M-12, B.Cu at (421.8, 101.8)
- added USB9: USB_C_Receptacle_USB2.0, Connector_USB:USB_C_Receptacle_HRO_TYPE-C-31-M-12, B.Cu at (155.1, 101.8)
- added Y1: 16MHz, Crystal:Crystal_SMD_2520-4Pin_2.5x2.0mm, F.Cu at (114.8, -17.0)
- added Y2: 16MHz, Crystal:Crystal_SMD_2520-4Pin_2.5x2.0mm, F.Cu at (116.3, 14.3)
- added Y3: 16MHz, Crystal:Crystal_SMD_2520-4Pin_2.5x2.0mm, F.Cu at (120.8, 14.3)
- added Y5: 16MHz, Crystal:Crystal_SMD_2520-4Pin_2.5x2.0mm, F.Cu at (120.8, 18.4)
- SW75: footprint Button_Switch_Keyboard:SW_Cherry_MX_2.00u_PCB -> Button_Switch_Keyboard:SW_Cherry_MX_2.25u_PCB
- USB1: renamed from J1; moved to B.Cu
- moved USB1 213.4 mm to (31.3, 101.8)
- moved RGB75 3.57 mm to (280.1, 212.5)
- moved SW34 3.57 mm to (270.4, 147.3)
- moved SW55 3.57 mm to (275.2, 166.4)
- moved SW91 3.57 mm to (263.3, 204.5)
- moved RGB36 3.57 mm to (149.1, 117.2)
- moved RGB38 3.57 mm to (187.2, 117.2)
- moved RGB39 3.57 mm to (206.3, 117.2)
- moved RGB40 3.57 mm to (225.3, 117.2)
- moved RGB41 3.57 mm to (244.4, 117.2)
- moved RGB42 3.57 mm to (149.1, 136.3)
- moved RGB44 3.57 mm to (187.2, 136.3)
- moved RGB45 3.57 mm to (206.3, 136.3)
- moved RGB46 3.57 mm to (225.3, 136.3)
- moved RGB47 3.57 mm to (244.4, 136.3)
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Other:
- board outline added: 476.2 x 129.8 mm

Commit message: added PCBs and plate
Parts:
- removed 7SD1, 7SD2: SA39-11EWA, Display_7Segment:Sx39-1xxxxx
Other:
- outline, holes or cut-outs redrawn
