File: KiCad Design/Project K+.kicad_pcb (KiCad board)
At the start: 2 copper layers, 476.2 x 129.8 mm, 364 parts, among them M3_SCREW_1 MountingHole, M3_SCREW_10 MountingHole, M3_SCREW_11 MountingHole, M3_SCREW_12 MountingHole, M3_SCREW_13 MountingHole, M3_SCREW_14 MountingHole, M3_SCREW_15 MountingHole, M3_SCREW_16 MountingHole, M3_SCREW_17 MountingHole, M3_SCREW_18 MountingHole, M3_SCREW_19 MountingHole, M3_SCREW_2 MountingHole, M3_SCREW_3 MountingHole, M3_SCREW_4 MountingHole, M3_SCREW_5 MountingHole, M3_SCREW_6 MountingHole, M3_SCREW_7 MountingHole, M3_SCREW_8 MountingHole, M3_SCREW_9 MountingHole, SW10 F5, SW100 LSPACE, SW101 RSPACE, SW102 ALTGR, SW103 FN, SW104 MENU, SW105 RCTRL, SW106 LEFT, SW107 DOWN, SW108 RIGHT, SW109 MACRO17, SW11 F6, SW110 MACRO18, SW111 MACRO19, SW112 MACRO20, SW12 F7, SW13 F8, SW14 F9, SW15 F10, SW16 F11, SW17 F12, SW18 PRTSCR, SW19 SCRLOCK, SW20 PAUSE, SW21 `, SW22 1, SW23 2, SW24 3, SW25 4, SW26 5, SW27 6, SW28 7, SW29 8, SW30 9, SW31 0, SW32 -, SW33 =, SW34 BACKSPACE, SW35 INSERT, SW36 HOME, SW37 PGUP, SW38 MACRO1, SW39 MACRO2, SW40 MACRO3, SW41 MACRO4, SW42 TAB, SW43 Q, SW44 W, SW45 E, SW46 R, SW47 T, SW48 Y, SW49 U, SW5 ESC, SW50 I, SW51 O, SW52 P, SW53 [, SW54 ], SW55 \, SW56 DEL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

Commit message: Switch to 75% layout
Parts:
- removed M3_SCREW_1, M3_SCREW_10, M3_SCREW_11, M3_SCREW_12, M3_SCREW_13, M3_SCREW_14, M3_SCREW_15, M3_SCREW_16, M3_SCREW_17, M3_SCREW_18, M3_SCREW_19, M3_SCREW_2, M3_SCREW_3, M3_SCREW_4, M3_SCREW_5, M3_SCREW_6, M3_SCREW_7, M3_SCREW_8, M3_SCREW_9: MountingHole, MountingHole:MountingHole_3.2mm_M3_Pad_Via
- removed SR1, SR10, SR11, SR12, SR13, SR14, SR15, SR16, SR17, SR18, SR19, SR2, SR20, SR21, SR22, SR3, SR4, SR5, SR6, SR7, SR8, SR9: 74HC165, Arduino_Pro_Micro:R-PDSO-G16
- removed SW109: MACRO17, Button_Switch_Keyboard:SW_Cherry_MX_1.00u_PCB
- removed SW110: MACRO18, Button_Switch_Keyboard:SW_Cherry_MX_1.00u_PCB
- removed SW111: MACRO19, Button_Switch_Keyboard:SW_Cherry_MX_1.00u_PCB
- removed SW112: MACRO20, Button_Switch_Keyboard:SW_Cherry_MX_1.00u_PCB
- removed U5: ATmega32U4-AU, Package_QFP:TQFP-44_10x10mm_P0.8mm
- added ARD1: ATmega32U4-A, Package_QFP:TQFP-44_10x10mm_P0.8mm, B.Cu at (46.0, 226.7)
- added ARD2: ATmega32U4-A, Package_QFP:TQFP-44_10x10mm_P0.8mm, F.Cu at (352.4, 253.6)
- added ARD3: ATmega32U4-A, Package_QFP:TQFP-44_10x10mm_P0.8mm, F.Cu at (418.4, 222.1)
- added ARD4: ATmega32U4-A, Package_QFP:TQFP-44_10x10mm_P0.8mm, F.Cu at (501.3, 222.6)
- added C16: 20pF, Capacitor_SMD:C_0603_1608Metric, F.Cu at (225.2, 174.6)
- added C18: 0.1uF, Capacitor_SMD:C_0603_1608Metric, F.Cu at (216.3, 179.6)
- added C19: 0.1uF, Capacitor_SMD:C_0603_1608Metric, F.Cu at (232.8, 177.1)
- added C22: 1uF, Capacitor_SMD:C_0603_1608Metric, F.Cu at (225.2, 172.1)
- added C24: 20pF, Capacitor_SMD:C_0603_1608Metric, F.Cu at (220.8, 177.1)
- added C26: 0.1uF, Capacitor_SMD:C_0603_1608Metric, F.Cu at (201.9, 184.0)
- added C27: 1uF, Capacitor_SMD:C_0603_1608Metric, F.Cu at (232.4, 179.6)
- added C28: 1uF, Capacitor_SMD:C_0603_1608Metric, F.Cu at (241.3, 171.5)
- added C29: 100n, Capacitor_SMD:C_0603_1608Metric, F.Cu at (515.5, 152.4)
- added C30: 100n, Capacitor_SMD:C_0603_1608Metric, F.Cu at (475.9, 190.4)
- added C31: 100n, Capacitor_SMD:C_0603_1608Metric, F.Cu at (455.9, 182.9)
- added C32: 100n, Capacitor_SMD:C_0603_1608Metric, F.Cu at (511.5, 157.4)
- added C33: 100n, Capacitor_SMD:C_0603_1608Metric, F.Cu at (511.5, 154.9)
- added C34: 100n, Capacitor_SMD:C_0603_1608Metric, F.Cu at (484.0, 185.4)
- added C35: 100n, Capacitor_SMD:C_0603_1608Metric, F.Cu at (459.9, 185.4)
- added C36: 100n, Capacitor_SMD:C_0603_1608Metric, F.Cu at (507.5, 154.9)
- added C37: 100n, Capacitor_SMD:C_0603_1608Metric, F.Cu at (467.9, 185.4)
- added C38: 100n, Capacitor_SMD:C_0603_1608Metric, F.Cu at (459.9, 182.9)
- added C39: 100n, Capacitor_SMD:C_0603_1608Metric, F.Cu at (484.0, 182.9)
- added C40: 100n, Capacitor_SMD:C_0603_1608Metric, F.Cu at (479.9, 187.9)
- added C41: 100n, Capacitor_SMD:C_0603_1608Metric, F.Cu at (463.9, 190.4)
- added C42: 100n, Capacitor_SMD:C_0603_1608Metric, F.Cu at (475.9, 187.9)
- added D10: G, Capacitor_SMD:C_0603_1608Metric, F.Cu at (201.9, 186.5)
- added D100: D, Diode_SMD:D_SOD-123F, B.Cu at (441.7, 354.8)
- added D101: D, Diode_SMD:D_SOD-123F, B.Cu at (479.8, 278.6)
- added D102: D, Diode_SMD:D_SOD-123F, B.Cu at (479.8, 297.7)
- added D103: D, Diode_SMD:D_SOD-123F, B.Cu at (479.8, 316.7)
- added D104: D, Diode_SMD:D_SOD-123F, B.Cu at (479.8, 335.8)
- added D105: D, Diode_SMD:D_SOD-123F, B.Cu at (479.8, 354.8)
- added D106: D, Diode_SMD:D_SOD-123F, B.Cu at (498.9, 278.6)
- added D107: D, Diode_SMD:D_SOD-123F, B.Cu at (498.9, 297.7)
- added D108: D, Diode_SMD:D_SOD-123F, B.Cu at (498.9, 316.7)
- added D109: D, Diode_SMD:D_SOD-123F, B.Cu at (498.9, 335.8)
- added D110: D, Diode_SMD:D_SOD-123F, B.Cu at (498.9, 354.8)
- added D111: D, Diode_SMD:D_SOD-123F, B.Cu at (517.9, 278.6)
- added D112: D, Diode_SMD:D_SOD-123F, B.Cu at (517.9, 297.7)
- added D113: D, Diode_SMD:D_SOD-123F, B.Cu at (517.9, 316.7)
- added D114: D, Diode_SMD:D_SOD-123F, B.Cu at (517.9, 335.8)
- added D115: D, Diode_SMD:D_SOD-123F, B.Cu at (517.9, 354.8)
- added D116: D, Diode_SMD:D_SOD-123F, B.Cu at (537.0, 278.6)
- added D117: D, Diode_SMD:D_SOD-123F, B.Cu at (537.0, 297.7)
- added D118: D, Diode_SMD:D_SOD-123F, B.Cu at (537.0, 316.7)
- added D119: D, Diode_SMD:D_SOD-123F, B.Cu at (537.0, 335.8)
- added D12: Y, Capacitor_SMD:C_0603_1608Metric, F.Cu at (208.7, 177.1)
- added D120: D, Diode_SMD:D_SOD-123F, B.Cu at (537.0, 354.8)
- added D121: D, Diode_SMD:D_SOD-123F, F.Cu at (529.6, 176.8)
- added D122: D, Diode_SMD:D_SOD-123F, F.Cu at (529.6, 173.4)
- added D123: D, Diode_SMD:D_SOD-123F, F.Cu at (535.1, 170.1)
- added D124: D, Diode_SMD:D_SOD-123F, F.Cu at (529.6, 170.1)
- added D13: D, Diode_SMD:D_SOD-123F, F.Cu at (79.8, 259.8)
- added D16: D, Diode_SMD:D_SOD-123F, F.Cu at (86.9, 316.9)
- added D17: D, Diode_SMD:D_SOD-123F, F.Cu at (91.7, 335.8)
- added D18: D, Diode_SMD:D_SOD-123F, F.Cu at (82.2, 354.8)
- added D19: D, Diode_SMD:D_SOD-123F, F.Cu at (98.8, 259.6)
- added D20: D, Diode_SMD:D_SOD-123F, F.Cu at (98.8, 278.6)
- added D21: D, Diode_SMD:D_SOD-123F, F.Cu at (108.3, 297.7)
- added D22: D, Diode_SMD:D_SOD-123F, F.Cu at (113.1, 316.7)
- added D23: D, Diode_SMD:D_SOD-123F, F.Cu at (122.6, 335.8)
- added D24: D, Diode_SMD:D_SOD-123F, F.Cu at (106.0, 354.8)
- added D25: D, Diode_SMD:D_SOD-123F, F.Cu at (117.9, 259.6)
- added D26: D, Diode_SMD:D_SOD-123F, F.Cu at (117.9, 278.6)
- added D27: D, Diode_SMD:D_SOD-123F, F.Cu at (127.4, 297.7)
- added D28: D, Diode_SMD:D_SOD-123F, F.Cu at (132.2, 316.7)
- added D29: D, Diode_SMD:D_SOD-123F, F.Cu at (141.7, 335.8)
- added D30: D, Diode_SMD:D_SOD-123F, F.Cu at (129.8, 354.8)
- added D31: D, Diode_SMD:D_SOD-123F, F.Cu at (136.9, 259.6)
- added D32: D, Diode_SMD:D_SOD-123F, F.Cu at (136.9, 278.6)
- added D33: D, Diode_SMD:D_SOD-123F, F.Cu at (146.4, 297.7)
- added D34: D, Diode_SMD:D_SOD-123F, F.Cu at (151.2, 316.7)
- added D35: D, Diode_SMD:D_SOD-123F, F.Cu at (160.7, 335.8)
- added D36: D, Diode_SMD:D_SOD-123F, F.Cu at (170.3, 354.8)
- added D37: D, Diode_SMD:D_SOD-123F, F.Cu at (156.0, 259.6)
- added D38: D, Diode_SMD:D_SOD-123F, F.Cu at (156.0, 278.6)
- added D39: D, Diode_SMD:D_SOD-123F, F.Cu at (165.5, 297.7)
- added D40: D, Diode_SMD:D_SOD-123F, F.Cu at (170.3, 316.7)
- added D41: D, Diode_SMD:D_SOD-123F, F.Cu at (177.4, 340.5)
- added D42: D, Diode_SMD:D_SOD-123F, F.Cu at (175.0, 259.6)
- added D43: D, Diode_SMD:D_SOD-123F, F.Cu at (175.0, 278.6)
- added D44: D, Diode_SMD:D_SOD-123F, F.Cu at (167.9, 291.7)
- added D45: D, Diode_SMD:D_SOD-123F, F.Cu at (172.6, 310.9)
- added D46: D, Diode_SMD:D_SOD-123F, F.Cu at (177.4, 253.6)
- added D47: D, Diode_SMD:D_SOD-123F, F.Cu at (177.4, 272.7)
- added D48: D, Diode_SMD:D_SOD-123F, B.Cu at (227.4, 297.7)
- added D49: D, Diode_SMD:D_SOD-123F, B.Cu at (236.9, 278.6)
- added D50: D, Diode_SMD:D_SOD-123F, B.Cu at (246.5, 297.7)
- added D51: D, Diode_SMD:D_SOD-123F, B.Cu at (232.2, 316.7)
- added D52: D, Diode_SMD:D_SOD-123F, B.Cu at (222.6, 335.8)
- added D53: D, Diode_SMD:D_SOD-123F, B.Cu at (236.9, 259.6)
- added D54: D, Diode_SMD:D_SOD-123F, B.Cu at (256.0, 278.6)
- added D55: D, Diode_SMD:D_SOD-123F, B.Cu at (265.5, 297.7)
- added D56: D, Diode_SMD:D_SOD-123F, B.Cu at (251.2, 316.7)
- added D57: D, Diode_SMD:D_SOD-123F, B.Cu at (241.7, 335.8)
- added D58: D, Diode_SMD:D_SOD-123F, B.Cu at (256.0, 259.6)
- added D59: D, Diode_SMD:D_SOD-123F, B.Cu at (275.0, 278.6)
- added D60: D, Diode_SMD:D_SOD-123F, B.Cu at (284.6, 297.7)
- added D61: D, Diode_SMD:D_SOD-123F, B.Cu at (270.3, 316.7)
- added D62: D, Diode_SMD:D_SOD-123F, B.Cu at (260.7, 335.8)
- added D63: D, Diode_SMD:D_SOD-123F, B.Cu at (253.6, 354.8)
- added D64: D, Diode_SMD:D_SOD-123F, B.Cu at (275.0, 259.6)
- added D65: D, Diode_SMD:D_SOD-123F, B.Cu at (294.1, 278.6)
- added D66: D, Diode_SMD:D_SOD-123F, B.Cu at (303.6, 297.7)
- added D67: D, Diode_SMD:D_SOD-123F, B.Cu at (289.3, 316.7)
- added D68: D, Diode_SMD:D_SOD-123F, B.Cu at (279.8, 335.8)
- added D69: D, Diode_SMD:D_SOD-123F, B.Cu at (296.5, 354.8)
- added D70: D, Diode_SMD:D_SOD-123F, B.Cu at (294.1, 259.6)
- added D71: D, Diode_SMD:D_SOD-123F, B.Cu at (313.1, 278.6)
- added D72: D, Diode_SMD:D_SOD-123F, B.Cu at (322.7, 297.7)
- added D73: D, Diode_SMD:D_SOD-123F, B.Cu at (308.4, 316.7)
- added D74: D, Diode_SMD:D_SOD-123F, B.Cu at (298.8, 335.8)
- added D75: D, Diode_SMD:D_SOD-123F, B.Cu at (320.3, 354.8)
- added D76: D, Diode_SMD:D_SOD-123F, B.Cu at (313.1, 259.6)
- added D77: D, Diode_SMD:D_SOD-123F, B.Cu at (332.2, 278.6)
- added D78: D, Diode_SMD:D_SOD-123F, B.Cu at (341.7, 297.7)
- added D79: D, Diode_SMD:D_SOD-123F, B.Cu at (327.4, 316.7)
- added D80: D, Diode_SMD:D_SOD-123F, B.Cu at (317.9, 335.8)
- added D81: D, Diode_SMD:D_SOD-123F, B.Cu at (344.1, 354.8)
- added D82: D, Diode_SMD:D_SOD-123F, B.Cu at (332.2, 259.6)
- added D83: D, Diode_SMD:D_SOD-123F, B.Cu at (360.8, 278.6)
- added D84: D, Diode_SMD:D_SOD-123F, B.Cu at (365.5, 297.7)
- added D85: D, Diode_SMD:D_SOD-123F, B.Cu at (358.4, 316.7)
- added D86: D, Diode_SMD:D_SOD-123F, B.Cu at (353.6, 335.8)
- added D87: D, Diode_SMD:D_SOD-123F, B.Cu at (367.9, 354.8)
- added D88: D, Diode_SMD:D_SOD-123F, B.Cu at (403.6, 278.6)
- added D89: D, Diode_SMD:D_SOD-123F, B.Cu at (403.6, 297.7)
- added D90: D, Diode_SMD:D_SOD-123F, B.Cu at (403.6, 316.7)
- added D91: D, Diode_SMD:D_SOD-123F, B.Cu at (403.6, 354.8)
- added D92: D, Diode_SMD:D_SOD-123F, B.Cu at (422.7, 278.6)
- added D93: D, Diode_SMD:D_SOD-123F, B.Cu at (422.7, 297.7)
- added D94: D, Diode_SMD:D_SOD-123F, B.Cu at (422.7, 316.7)
- added D95: D, Diode_SMD:D_SOD-123F, B.Cu at (422.7, 335.8)
- added D96: D, Diode_SMD:D_SOD-123F, B.Cu at (422.7, 354.8)
- added D97: D, Diode_SMD:D_SOD-123F, B.Cu at (441.7, 278.6)
- added D98: D, Diode_SMD:D_SOD-123F, B.Cu at (441.7, 297.7)
- added D99: D, Diode_SMD:D_SOD-123F, B.Cu at (441.7, 316.7)
- added P1: TESTPAD, TestPoint:TestPoint_Pad_2.0x2.0mm, F.Cu at (537.0, 161.3)
- added P10: TESTPAD, TestPoint:TestPoint_Pad_2.0x2.0mm, F.Cu at (528.9, 153.2)
- added P11: TESTPAD, TestPoint:TestPoint_Pad_2.0x2.0mm, F.Cu at (528.9, 157.2)
- added P12: TESTPAD, TestPoint:TestPoint_Pad_2.0x2.0mm, F.Cu at (533.0, 153.2)
- added P2: TESTPAD, TestPoint:TestPoint_Pad_2.0x2.0mm, F.Cu at (541.1, 157.2)
- added P3: TESTPAD, TestPoint:TestPoint_Pad_2.0x2.0mm, F.Cu at (537.0, 153.2)
- added P4: TESTPAD, TestPoint:TestPoint_Pad_2.0x2.0mm, F.Cu at (541.1, 153.2)
- added P5: TESTPAD, TestPoint:TestPoint_Pad_2.0x2.0mm, F.Cu at (537.0, 157.2)
- added P6: TESTPAD, TestPoint:TestPoint_Pad_2.0x2.0mm, F.Cu at (533.0, 157.2)
- added P7: TESTPAD, TestPoint:TestPoint_Pad_2.0x2.0mm, F.Cu at (528.9, 161.3)
- added P8: TESTPAD, TestPoint:TestPoint_Pad_2.0x2.0mm, F.Cu at (541.1, 161.3)
- added P9: TESTPAD, TestPoint:TestPoint_Pad_2.0x2.0mm, F.Cu at (533.0, 161.3)
- added R100: 10K, Resistor_SMD:R_0603_1608Metric, F.Cu at (479.9, 182.9)
- added R101: 10K, Resistor_SMD:R_0603_1608Metric, F.Cu at (459.9, 187.9)
- added R46: 56K, Resistor_SMD:R_0603_1608Metric, B.Cu at (242.9, 239.3)
- added R48: 680R, Resistor_SMD:R_0603_1608Metric, B.Cu at (491.7, 230.3)
- added R50: 680R, Resistor_SMD:R_0603_1608Metric, B.Cu at (267.8, 230.3)
- added R52: 22R, Resistor_SMD:R_0603_1608Metric, F.Cu at (237.2, 173.0)
- added R54: 22R, Resistor_SMD:R_0603_1608Metric, F.Cu at (201.9, 191.5)
- added R56: 10K, Resistor_SMD:R_0603_1608Metric, F.Cu at (201.9, 189.0)
- added R58: 330R, Resistor_SMD:R_0603_1608Metric, F.Cu at (233.2, 173.0)
- added R59: 330R, Resistor_SMD:R_0603_1608Metric, F.Cu at (229.2, 172.1)
- added R62: 1K, Resistor_SMD:R_0603_1608Metric, F.Cu at (213.2, 172.1)
- added R63: 330R, Resistor_SMD:R_0603_1608Metric, F.Cu at (208.3, 179.6)
- added R64: 22R, Resistor_SMD:R_0603_1608Metric, F.Cu at (224.3, 179.6)
- added R65: 22R, Resistor_SMD:R_0603_1608Metric, F.Cu at (212.3, 179.6)
- added R66: 10K, Resistor_SMD:R_0603_1608Metric, F.Cu at (220.3, 179.6)
- added R67: 330R, Resistor_SMD:R_0603_1608Metric, F.Cu at (213.2, 174.6)
- added R68: 1K, Resistor_SMD:R_0603_1608Metric, F.Cu at (229.2, 174.6)
- added R69: 330R, Resistor_SMD:R_0603_1608Metric, F.Cu at (228.3, 179.6)
- added R70: 10K, Resistor_SMD:R_0603_1608Metric, B.Cu at (65.5, 355.2)
- added R71: 10K, Resistor_SMD:R_0603_1608Metric, B.Cu at (89.3, 354.8)
- added R72: 10K, Resistor_SMD:R_0603_1608Metric, B.Cu at (113.1, 354.8)
- added R73: 10K, Resistor_SMD:R_0603_1608Metric, B.Cu at (153.6, 354.4)
- added R74: 10K, Resistor_SMD:R_0603_1608Metric, B.Cu at (163.1, 336.1)
- added R75: 10K, Resistor_SMD:R_0603_1608Metric, B.Cu at (172.6, 316.7)
- added R76: 10K, Resistor_SMD:R_0603_1608Metric, B.Cu at (177.7, 260.3)
- added R77: 10K, Resistor_SMD:R_0603_1608Metric, F.Cu at (373.4, 198.1)
- added R78: 10K, Resistor_SMD:R_0603_1608Metric, F.Cu at (185.0, 200.0)
- added R79: 10K, Resistor_SMD:R_0603_1608Metric, F.Cu at (362.7, 157.0)
- added R80: 10K, Resistor_SMD:R_0603_1608Metric, F.Cu at (362.7, 154.5)
- added R81: 10K, Resistor_SMD:R_0603_1608Metric, F.Cu at (164.9, 200.0)
- added R82: 10K, Resistor_SMD:R_0603_1608Metric, F.Cu at (362.7, 147.0)
- added R83: 10K, Resistor_SMD:R_0603_1608Metric, F.Cu at (362.7, 152.0)
- added R84: 10K, Resistor_SMD:R_0603_1608Metric, F.Cu at (362.7, 162.1)
- added R85: 10K, Resistor_SMD:R_0603_1608Metric, F.Cu at (177.0, 200.0)
- added R86: 10K, Resistor_SMD:R_0603_1608Metric, F.Cu at (173.0, 200.0)
- added R87: 10K, Resistor_SMD:R_0603_1608Metric, F.Cu at (362.7, 144.5)
- added R88: 10K, Resistor_SMD:R_0603_1608Metric, F.Cu at (373.4, 195.6)
- added R89: 10K, Resistor_SMD:R_0603_1608Metric, F.Cu at (373.4, 185.5)
- added R90: 10K, Resistor_SMD:R_0603_1608Metric, F.Cu at (362.7, 159.6)
- added R91: 10K, Resistor_SMD:R_0603_1608Metric, F.Cu at (362.7, 149.5)
- added R92: 10K, Resistor_SMD:R_0603_1608Metric, F.Cu at (451.9, 190.4)
- added R93: 10K, Resistor_SMD:R_0603_1608Metric, F.Cu at (455.9, 187.9)
- added R94: 10K, Resistor_SMD:R_0603_1608Metric, F.Cu at (451.9, 185.4)
- added R95: 220R, Resistor_SMD:R_0603_1608Metric, F.Cu at (451.9, 182.9)
- added R96: 10K, Resistor_SMD:R_0603_1608Metric, F.Cu at (507.5, 159.9)
- added R97: 10K, Resistor_SMD:R_0603_1608Metric, F.Cu at (515.5, 154.9)
- added R98: 10K, Resistor_SMD:R_0603_1608Metric, F.Cu at (479.9, 185.4)
- added R99: 10K, Resistor_SMD:R_0603_1608Metric, F.Cu at (471.9, 187.9)
- added SW1: ESC, Button_Switch_Keyboard:SW_Cherry_MX_1.00u_PCB, F.Cu at (68.9, 259.9)
- added SW2: `, Button_Switch_Keyboard:SW_Cherry_MX_1.00u_PCB, F.Cu at (68.9, 278.9)
- added SW3: TAB, Button_Switch_Keyboard:SW_Cherry_MX_1.50u_PCB, F.Cu at (73.7, 298.0)
- added SW4: CAPS, Button_Switch_Keyboard:SW_Cherry_MX_1.75u_PCB, F.Cu at (76.0, 317.0)
- added U4: GL850G-HHGXX(SSOP-28), Package_SO:SSOP-28_5.3x10.2mm_P0.65mm, B.Cu at (259.6, 235.7)
- added USB10: USB_C_Receptacle_USB2.0, Connector_USB:USB_C_Receptacle_Palconn_UTC16-G, B.Cu at (344.1, 233.2)
- added USB11: USB_A, Connector_USB:USB_A_Molex_67643_Horizontal, B.Cu at (357.3, 241.1)
- added USB12: USB_A, Connector_USB:USB_A_Molex_67643_Horizontal, B.Cu at (323.9, 241.1)
- added USB2: USB_C_Receptacle_USB2.0, Connector_USB:USB_C_Receptacle_Palconn_UTC16-G, B.Cu at (433.4, 233.4)
- added USB6: USB_A, Connector_USB:USB_A_Molex_67643_Horizontal, B.Cu at (146.5, 241.1)
- added Y4: 12MHz, Crystal:Crystal_SMD_2520-4Pin_2.5x2.0mm, B.Cu at (491.7, 235.1)
- added Y6: 16MHz, Crystal:Crystal_SMD_2520-4Pin_2.5x2.0mm, F.Cu at (123.0, 211.3)
- added Y7: 16MHz, Crystal:Crystal_SMD_2520-4Pin_2.5x2.0mm, F.Cu at (118.5, 211.3)
- added Y8: 16MHz, Crystal:Crystal_SMD_2520-4Pin_2.5x2.0mm, F.Cu at (113.8, 211.3)
- C10, C11, C2, C3, C8, C9, R22, R23, Y1: moved to B.Cu
- C12, C13: value 0.1uF -> 20pF; moved to B.Cu
- C14, C15, C17, C25: value 1uF -> 20pF
- C20, C21: value 20pF -> 1uF
- C23: value 0.1uF -> 1uF
- C6, C7: value 1uF -> 20pF; moved to B.Cu
- D14: value G -> D; footprint Capacitor_SMD:C_0603_1608Metric -> Diode_SMD:D_SOD-123F
- D15: value Y -> D; footprint Capacitor_SMD:C_0603_1608Metric -> Diode_SMD:D_SOD-123F
- D4, D5: value LED -> G
- D6, D8: value G -> LED
- R10: value 5.1K -> 220R
- R11, R13, R14, R16, R17, R19, R2, R20, R3, R4, R5, R7, R8: value 5.1K -> 10K
- R12, R15, R18, R21, R6, R9: value 220R -> 10K
- R30, R31, R47: value 1K -> 56K; moved to B.Cu
- R32, R33: value 10K -> 5.1K; moved to B.Cu
- R34, R35: value 5.1K -> 56K; moved to B.Cu
- R36, R37, R51: value 5.1K -> 680R; moved to B.Cu
- R38, R39: value 22R -> 680R; moved to B.Cu
- R40, R41: value 22R -> 5.1K; moved to B.Cu
- R42, R43: value 330R -> 56K; moved to B.Cu
- R44, R45: value 330R -> 5.1K; moved to B.Cu
- R49: value 10K -> 680R; moved to B.Cu
- R53: value 5.1K -> 22R
- R57: value 22R -> 10K
- R60: value 330R -> 1K
- RE1, RE2, RE3, RE4, RE5, RE6, RE7: value (none) -> ~
- SW10: value F5 -> A
- SW100: value LSPACE -> MACRO7; footprint Cherry_MX_SMD:SW_Cherry_MX_3.00u_PCB -> Button_Switch_Keyboard:SW_Cherry_MX_1.00u_PCB
- SW101: value RSPACE -> MACRO11; footprint Cherry_MX_SMD:SW_Cherry_MX_3.25u_PCB -> Button_Switch_Keyboard:SW_Cherry_MX_1.00u_PCB
- SW102: value ALTGR -> MACRO15; footprint Button_Switch_Keyboard:SW_Cherry_MX_1.25u_PCB -> Button_Switch_Keyboard:SW_Cherry_MX_1.00u_PCB
- SW103: value FN -> MACRO19; footprint Button_Switch_Keyboard:SW_Cherry_MX_1.25u_PCB -> Button_Switch_Keyboard:SW_Cherry_MX_1.00u_PCB
- SW104: value MENU -> MACRO4; footprint Button_Switch_Keyboard:SW_Cherry_MX_1.25u_PCB -> Button_Switch_Keyboard:SW_Cherry_MX_1.00u_PCB
- SW105: value RCTRL -> MACRO8; footprint Button_Switch_Keyboard:SW_Cherry_MX_1.25u_PCB -> Button_Switch_Keyboard:SW_Cherry_MX_1.00u_PCB
- SW106: value LEFT -> MACRO12
- SW107: value DOWN -> MACRO16
- SW108: value RIGHT -> MACRO20
- SW11: value F6 -> Z
- SW12: value F7 -> OS; footprint Button_Switch_Keyboard:SW_Cherry_MX_1.00u_PCB -> Button_Switch_Keyboard:SW_Cherry_MX_1.25u_PCB
- SW13: value F8 -> F2
- SW14: value F9 -> 2
- SW15: value F10 -> W
- SW16: value F11 -> S
- SW17: value F12 -> X
- SW18: value PRTSCR -> L_ALT; footprint Button_Switch_Keyboard:SW_Cherry_MX_1.00u_PCB -> Button_Switch_Keyboard:SW_Cherry_MX_1.25u_PCB
- SW19: value SCRLOCK -> F3
- SW20: value PAUSE -> 3
- SW21: value ` -> E
- SW22: value 1 -> D
- SW23: value 2 -> C
- SW24: value 3 -> L_SPACE; footprint Button_Switch_Keyboard:SW_Cherry_MX_1.00u_PCB -> Button_Switch_Keyboard:SW_Cherry_MX_2.25u_PCB
- SW25: value 4 -> F4
- SW26: value 5 -> 4
- SW27: value 6 -> R
- SW28: value 7 -> F
- SW29: value 8 -> V
- SW30: value 9 -> F5
- SW31: value 0 -> 5
- SW32: value - -> T
- SW33: value = -> G
- SW34: value BACKSPACE -> F6; footprint Button_Switch_Keyboard:SW_Cherry_MX_2.00u_PCB -> Button_Switch_Keyboard:SW_Cherry_MX_1.00u_PCB
- SW35: value INSERT -> 6
- SW36: value HOME -> Y
- SW37: value PGUP -> 7
- SW38: value MACRO1 -> U
- SW39: value MACRO2 -> H
- SW40: value MACRO3 -> B
- SW41: value MACRO4 -> F7
- SW42: value TAB -> 8; footprint Button_Switch_Keyboard:SW_Cherry_MX_1.50u_PCB -> Button_Switch_Keyboard:SW_Cherry_MX_1.00u_PCB
- SW43: value Q -> I
- SW44: value W -> J
- SW45: value E -> N
- SW46: value R -> F8
- SW47: value T -> 9
- SW48: value Y -> O
- SW49: value U -> K
- SW5: value ESC -> L_SHIFT; footprint Button_Switch_Keyboard:SW_Cherry_MX_1.00u_PCB -> Button_Switch_Keyboard:SW_Cherry_MX_2.25u_PCB
- SW50: value I -> M
- SW51: value O -> R_SPACE; footprint Button_Switch_Keyboard:SW_Cherry_MX_1.00u_PCB -> Button_Switch_Keyboard:SW_Cherry_MX_2.25u_PCB
- SW52: value P -> F9
- SW53: value [ -> 0
- SW54: value ] -> P
- SW55: value \ -> L; footprint Button_Switch_Keyboard:SW_Cherry_MX_1.50u_PCB -> Button_Switch_Keyboard:SW_Cherry_MX_1.00u_PCB
- SW56: value DEL -> ,
- SW57: value END -> R_ALT; footprint Button_Switch_Keyboard:SW_Cherry_MX_1.00u_PCB -> Button_Switch_Keyboard:SW_Cherry_MX_1.25u_PCB
- SW58: value PGDN -> F10
- SW59: value MACRO5 -> -
- SW6: value F1 -> L_CTRL; footprint Button_Switch_Keyboard:SW_Cherry_MX_1.00u_PCB -> Button_Switch_Keyboard:SW_Cherry_MX_1.25u_PCB
- SW60: value MACRO6 -> [
- SW61: value MACRO7 -> ;
- SW62: value MACRO8 -> .
- SW63: value CAPSLOCK -> FN; footprint Button_Switch_Keyboard:SW_Cherry_MX_1.75u_PCB -> Button_Switch_Keyboard:SW_Cherry_MX_1.25u_PCB
- SW64: value A -> F11
- SW65: value S -> =
- SW66: value D -> ]
- SW67: value F -> '
- SW68: value G -> /
- SW69: value H -> MENU; footprint Button_Switch_Keyboard:SW_Cherry_MX_1.00u_PCB -> Button_Switch_Keyboard:SW_Cherry_MX_1.25u_PCB
- SW7: value F2 -> F1
- SW70: value J -> F12
- SW71: value K -> BACKSPACE; footprint Button_Switch_Keyboard:SW_Cherry_MX_1.00u_PCB -> Button_Switch_Keyboard:SW_Cherry_MX_2.00u_PCB
- SW72: value L -> \; footprint Button_Switch_Keyboard:SW_Cherry_MX_1.00u_PCB -> Button_Switch_Keyboard:SW_Cherry_MX_1.50u_PCB
- SW73: value ; -> RETURN; footprint Button_Switch_Keyboard:SW_Cherry_MX_1.00u_PCB -> Button_Switch_Keyboard:SW_Cherry_MX_2.25u_PCB
- SW74: value ' -> R_SHIFT; footprint Button_Switch_Keyboard:SW_Cherry_MX_1.00u_PCB -> Button_Switch_Keyboard:SW_Cherry_MX_2.75u_PCB
- SW75: value RETURN -> R_CTRL; footprint Button_Switch_Keyboard:SW_Cherry_MX_2.25u_PCB -> Button_Switch_Keyboard:SW_Cherry_MX_1.25u_PCB
- SW76: value MACRO9 -> PRTSCR
- SW77: value MACRO10 -> INSERT
- SW78: value MACRO11 -> DELETE
- SW79: value MACRO12 -> LEFT
- SW8: value F3 -> 1
- SW80: value LSHIFT -> SCRLOCK; footprint Button_Switch_Keyboard:SW_Cherry_MX_2.25u_PCB -> Button_Switch_Keyboard:SW_Cherry_MX_1.00u_PCB
- SW81: value Z -> HOME
- SW82: value X -> END
- SW83: value C -> UP
- SW84: value V -> DOWN
- SW85: value B -> PAUSE
- SW86: value N -> PGUP
- SW87: value M -> PGDN
- SW88: value , -> RIGHT
- SW89: value . -> MACRO1
- SW9: value F4 -> Q
- SW90: value / -> MACRO5
- SW91: value RSHIFT -> MACRO9; footprint Button_Switch_Keyboard:SW_Cherry_MX_2.75u_PCB -> Button_Switch_Keyboard:SW_Cherry_MX_1.00u_PCB
- SW92: value UP -> MACRO13
- SW93: value MACRO13 -> MACRO17
- SW94: value MACRO14 -> MACRO2
- SW95: value MACRO15 -> MACRO6
- SW96: value MACRO16 -> MACRO10
- SW97: value LCTRL -> MACRO14; footprint Button_Switch_Keyboard:SW_Cherry_MX_1.25u_PCB -> Button_Switch_Keyboard:SW_Cherry_MX_1.00u_PCB
- SW98: value OS -> MACRO18; footprint Button_Switch_Keyboard:SW_Cherry_MX_1.25u_PCB -> Button_Switch_Keyboard:SW_Cherry_MX_1.00u_PCB
- SW99: value ALT -> MACRO3; footprint Button_Switch_Keyboard:SW_Cherry_MX_1.25u_PCB -> Button_Switch_Keyboard:SW_Cherry_MX_1.00u_PCB
- U1, U2, U3: value ATmega32U4-AU -> GL850G-HHGXX(SSOP-28); footprint Package_QFP:TQFP-44_10x10mm_P0.8mm -> Package_SO:SSOP-28_5.3x10.2mm_P0.65mm; moved to B.Cu
- USB1, USB3, USB4, USB7, USB8, USB9: footprint Connector_USB:USB_C_Receptacle_HRO_TYPE-C-31-M-12 -> Connector_USB:USB_C_Receptacle_Palconn_UTC16-G
- USB5: value USB_C_Receptacle_USB2.0 -> USB_A; footprint Connector_USB:USB_C_Receptacle_HRO_TYPE-C-31-M-12 -> Connector_USB:USB_A_Molex_67643_Horizontal
- Y2, Y3, Y5: value 16MHz -> 12MHz; moved to B.Cu
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Connections:
- net RGB2_OUT renamed RGB_OUT_R
- net RGB3_OUT renamed RGB_OUT_A
- net RGB_OUT renamed RGB_OUT_N
- C1 pad 1: +5V -> C0_A
- C14 pad 1: Net-(C14-Pad1) -> Net-(ARD2-Pad17)
- C15 pad 1: Net-(C15-Pad1) -> Net-(ARD3-Pad17)
- C17 pad 1: +5V -> Net-(ARD3-Pad16)
- C2 pad 1: Net-(C2-Pad1) -> Net-(ARD1-Pad17)
- C2 pad 2: Net-(C2-Pad2) -> GND
- C20 pad 1: Net-(C20-Pad1) -> Net-(ARD2-Pad6)
- C21 pad 1: Net-(C21-Pad1) -> Net-(ARD3-Pad6)
- C23 pad 1: Net-(C23-Pad1) -> C0_A
- C3 pad 1: Net-(C3-Pad1) -> Net-(ARD1-Pad16)
- C4 pad 1: Net-(C4-Pad1) -> Net-(ARD1-Pad42)
- C5 pad 1: Net-(C5-Pad1) -> Net-(ARD1-Pad6)
- C6 pad 1: +5V -> Net-(C6-Pad1)
- C7 pad 1: +5V -> Net-(C7-Pad1)
- D14 pad 1: VCC -> R1_L
- D15 pad 1: VCC -> R2_L
- D2 pad 1: VCC -> C0_A
- D3 pad 1: VCC -> C0_A
- D4 pad 1: GND -> VCC
- D5 pad 1: GND -> VCC
- D6 pad 1: VCC -> GND
- D8 pad 1: VCC -> GND
- R1 pad 1: SW4 -> SW1
- R10 pad 1: A3 -> SW3
- R10 pad 2: +5V -> Net-(R10-Pad2)
- R11 pad 1: +5V -> B1
- R11 pad 2: B3 -> Net-(RE1-PadB)
- R12 pad 1: SW1 -> B3
- R13 pad 1: A4 -> B5
- R13 pad 2: +5V -> Net-(R13-Pad2)
- R14 pad 1: +5V -> B7
- R14 pad 2: B4 -> Net-(R14-Pad2)
- R15 pad 1: SW4 -> C0_A
- R15 pad 2: Net-(R15-Pad2) -> Net-(RE1-PadB)
- R16 pad 1: A5 -> C0_A
- R16 pad 2: +5V -> Net-(R12-Pad2)
- R17 pad 1: +5V -> C0_A
- R17 pad 2: B5 -> Net-(R13-Pad2)
- R18 pad 1: SW3 -> C0_A
- R18 pad 2: Net-(R18-Pad2) -> Net-(R14-Pad2)
- R19 pad 1: A6 -> C0_A
- R19 pad 2: +5V -> Net-(R19-Pad2)
- R2 pad 1: GND -> C0_A
- R2 pad 2: Net-(R2-Pad2) -> Net-(RE1-PadA)
- R20 pad 1: +5V -> C0_A
- R20 pad 2: B6 -> Net-(R20-Pad2)
- R21 pad 1: SW2 -> C0_A
- R22 pad 1: A7 -> Net-(R22-Pad1)
- R22 pad 2: +5V -> GND
- R23 pad 1: +5V -> Net-(R23-Pad1)
- R23 pad 2: B7 -> GND
- R24 pad 1: +5V -> C0_A
- R25 pad 1: +5V -> C0_A
- R25 pad 2: Net-(R25-Pad2) -> Net-(ARD1-Pad13)
- R26 pad 1: Net-(R26-Pad1) -> Net-(ARD1-Pad4)
- R26 pad 2: D+_ATMEGA32U4 -> L_D+
- R27 pad 1: D-_ATMEGA32U4 -> L_D-
- R27 pad 2: Net-(R27-Pad2) -> Net-(ARD1-Pad3)
- R28 pad 1: Net-(R28-Pad1) -> Net-(ARD1-Pad22)
- R29 pad 1: D14 -> Net-(ARD1-Pad8)
- R3 pad 1: Net-(R3-Pad1) -> C0_A
- R3 pad 2: GND -> Net-(R3-Pad2)
- R30 pad 1: +5V -> Net-(R30-Pad1)
- R30 pad 2: Net-(D4-Pad2) -> C0_A
- R31 pad 1: +5V -> Net-(R31-Pad1)
- R31 pad 2: Net-(D5-Pad2) -> C0_A
- R32 pad 1: +5V -> Net-(R32-Pad1)
- R32 pad 2: Net-(R32-Pad2) -> GND
- R33 pad 1: +5V -> Net-(R33-Pad1)
- R33 pad 2: Net-(R33-Pad2) -> GND
- R34 pad 1: GND -> Net-(R34-Pad1)
- R34 pad 2: Net-(R34-Pad2) -> C0_A
- R35 pad 1: GND -> Net-(R35-Pad1)
- R35 pad 2: Net-(R35-Pad2) -> C0_A
- R37 pad 2: GND -> C0_A
- R38 pad 2: Net-(R38-Pad2) -> GND
- R39 pad 2: Net-(R39-Pad2) -> C0_A
- R4 pad 1: A1 -> C0_A
- R4 pad 2: +5V -> Net-(R4-Pad2)
- R40 pad 2: Net-(R40-Pad2) -> GND
- R41 pad 2: Net-(R41-Pad2) -> GND
- R42 pad 2: Net-(D6-Pad2) -> C0_A
- R43 pad 1: D14 -> Net-(R43-Pad1)
- R43 pad 2: Net-(D7-Pad2) -> C0_A
- R44 pad 2: Net-(D8-Pad2) -> GND
- R45 pad 1: D14 -> Net-(R45-Pad1)
- R45 pad 2: Net-(D9-Pad2) -> GND
- R47 pad 1: +5V -> Net-(R47-Pad1)
- R47 pad 2: Net-(D11-Pad2) -> C0_A
- R49 pad 1: +5V -> Net-(R49-Pad1)
- R49 pad 2: Net-(R49-Pad2) -> C0_A
- R5 pad 1: +5V -> C0_A
- R5 pad 2: B1 -> Net-(R5-Pad2)
- R51 pad 1: GND -> Net-(R51-Pad1)
- R51 pad 2: Net-(R51-Pad2) -> C0_A
- R53 pad 1: Net-(R53-Pad1) -> D-_R
- R53 pad 2: GND -> Net-(ARD2-Pad3)
- R55 pad 1: Net-(R55-Pad1) -> D-_N
- R55 pad 2: Net-(R55-Pad2) -> Net-(ARD3-Pad3)
- R57 pad 1: Net-(R57-Pad1) -> C0_A
- R6 pad 1: SW3 -> A1
- R6 pad 2: Net-(R6-Pad2) -> Net-(RE1-PadA)
- R60 pad 1: Net-(R60-Pad1) -> C0_A
- R60 pad 2: Net-(D14-Pad2) -> Net-(D6-Pad2)
- R61 pad 1: D14 -> Net-(ARD2-Pad8)
- R61 pad 2: Net-(D15-Pad2) -> Net-(D7-Pad2)
- R7 pad 1: A2 -> A3
- R7 pad 2: +5V -> Net-(R3-Pad2)
- R8 pad 1: +5V -> A5
- R8 pad 2: B2 -> Net-(R4-Pad2)
- R9 pad 1: SW2 -> A7
- R9 pad 2: Net-(R9-Pad2) -> Net-(R5-Pad2)
- RE1 pad A: A1 -> Net-(RE1-PadA)
- RE1 pad B: B1 -> Net-(RE1-PadB)
- RE2 pad A: A2 -> Net-(R3-Pad2)
- RE2 pad B: B2 -> Net-(R12-Pad2)
- RE2 pad S1: Net-(R6-Pad2) -> Net-(R10-Pad2)
- RE3 pad A: A3 -> Net-(R4-Pad2)
- RE3 pad B: B3 -> Net-(R13-Pad2)
- RE3 pad S1: Net-(R9-Pad2) -> SW5_1
- RE3 pad S2: GND -> SW5_2
- RE4 pad A: A4 -> Net-(R5-Pad2)
- RE4 pad B: B4 -> Net-(R14-Pad2)
- RE4 pad S1: Net-(R12-Pad2) -> SW7_1
- RE4 pad S2: GND -> SW7_2
- RE5 pad A: A5 -> Net-(R19-Pad2)
- RE5 pad B: B5 -> Net-(R96-Pad2)
- RE5 pad S1: Net-(R15-Pad2) -> Net-(R95-Pad2)
- RE6 pad A: A6 -> Net-(R20-Pad2)
- RE6 pad B: B6 -> Net-(R100-Pad2)
- RE6 pad S1: Net-(R18-Pad2) -> SW4_1
- RE6 pad S2: GND -> SW4_2
- RE7 pad A: A7 -> Net-(R21-Pad2)
- RE7 pad B: B7 -> Net-(R101-Pad2)
- RE7 pad S1: Net-(R21-Pad2) -> SW6_1
- RE7 pad S2: GND -> SW6_2
- RGB1 pad 1: +5V -> C0_A
- RGB1 pad 4: RGB_IN -> RGB_IN_L
- RGB10 pad 1: +5V -> C0_A
- RGB100 pad 1: +5V -> C0_A
- RGB101 pad 1: +5V -> C0_A
- RGB102 pad 1: +5V -> C0_A
- RGB103 pad 1: +5V -> C0_A
- RGB104 pad 1: +5V -> C0_A
- RGB105 pad 1: +5V -> C0_A
- RGB106 pad 1: +5V -> C0_A
- RGB107 pad 1: +5V -> C0_A
- RGB108 pad 1: +5V -> C0_A
- RGB11 pad 1: +5V -> C0_A
- RGB12 pad 1: +5V -> C0_A
- RGB13 pad 1: +5V -> C0_A
- RGB14 pad 1: +5V -> C0_A
- RGB15 pad 1: +5V -> C0_A
- RGB16 pad 1: +5V -> C0_A
- RGB17 pad 1: +5V -> C0_A
- RGB18 pad 1: +5V -> C0_A
- RGB19 pad 1: +5V -> C0_A
- RGB2 pad 1: +5V -> C0_A
- RGB20 pad 1: +5V -> C0_A
- RGB21 pad 1: +5V -> C0_A
- RGB22 pad 1: +5V -> C0_A
- RGB23 pad 1: +5V -> C0_A
- RGB24 pad 1: +5V -> C0_A
- RGB25 pad 1: +5V -> C0_A
- RGB26 pad 1: +5V -> C0_A
- RGB27 pad 1: +5V -> C0_A
- RGB28 pad 1: +5V -> C0_A
- RGB29 pad 1: +5V -> C0_A
- RGB3 pad 1: +5V -> C0_A
- RGB30 pad 1: +5V -> C0_A
- RGB31 pad 1: +5V -> C0_A
- RGB32 pad 1: +5V -> C0_A
- RGB33 pad 1: +5V -> C0_A
- RGB34 pad 1: +5V -> C0_A
- RGB35 pad 1: +5V -> C0_A
- RGB35 pad 2: RGB1_OUT -> RGB_OUT_L
- RGB36 pad 1: +5V -> C0_A
- RGB36 pad 4: RGB1_IN -> RGB_IN_R
- RGB37 pad 1: +5V -> C0_A
- RGB38 pad 1: +5V -> C0_A
- RGB39 pad 1: +5V -> C0_A
- RGB4 pad 1: +5V -> C0_A
- RGB40 pad 1: +5V -> C0_A
- RGB41 pad 1: +5V -> C0_A
- RGB42 pad 1: +5V -> C0_A
- RGB43 pad 1: +5V -> C0_A
- RGB44 pad 1: +5V -> C0_A
- RGB45 pad 1: +5V -> C0_A
- RGB46 pad 1: +5V -> C0_A
- RGB47 pad 1: +5V -> C0_A
- RGB48 pad 1: +5V -> C0_A
- RGB49 pad 1: +5V -> C0_A
- RGB5 pad 1: +5V -> C0_A
- RGB50 pad 1: +5V -> C0_A
- RGB51 pad 1: +5V -> C0_A
- RGB52 pad 1: +5V -> C0_A
- RGB53 pad 1: +5V -> C0_A
- RGB54 pad 1: +5V -> C0_A
- RGB55 pad 1: +5V -> C0_A
- RGB56 pad 1: +5V -> C0_A
- RGB57 pad 1: +5V -> C0_A
- RGB58 pad 1: +5V -> C0_A
- RGB59 pad 1: +5V -> C0_A
- RGB6 pad 1: +5V -> C0_A
- RGB60 pad 1: +5V -> C0_A
- RGB61 pad 1: +5V -> C0_A
- RGB62 pad 1: +5V -> C0_A
- RGB63 pad 1: +5V -> C0_A
- RGB64 pad 1: +5V -> C0_A
- RGB65 pad 1: +5V -> C0_A
- RGB66 pad 1: +5V -> C0_A
- RGB67 pad 1: +5V -> C0_A
- RGB68 pad 1: +5V -> C0_A
- RGB69 pad 1: +5V -> C0_A
- RGB7 pad 1: +5V -> C0_A
- RGB70 pad 1: +5V -> C0_A
- RGB71 pad 1: +5V -> C0_A
- RGB72 pad 1: +5V -> C0_A
- RGB73 pad 1: +5V -> C0_A
- RGB74 pad 1: +5V -> C0_A
- RGB75 pad 1: +5V -> C0_A
- RGB76 pad 1: +5V -> C0_A
- RGB76 pad 4: RGB2_IN -> RGB_IN_A
- RGB77 pad 1: +5V -> C0_A
- RGB78 pad 1: +5V -> C0_A
- RGB79 pad 1: +5V -> C0_A
- RGB8 pad 1: +5V -> C0_A
- RGB80 pad 1: +5V -> C0_A
- RGB81 pad 1: +5V -> C0_A
- RGB82 pad 1: +5V -> C0_A
- RGB83 pad 1: +5V -> C0_A
- RGB84 pad 1: +5V -> C0_A
- RGB85 pad 1: +5V -> C0_A
- RGB86 pad 1: +5V -> C0_A
- RGB87 pad 1: +5V -> C0_A
- RGB88 pad 1: +5V -> C0_A
- RGB89 pad 1: +5V -> C0_A
- RGB89 pad 4: RGB3_IN -> RGB_IN_N
- RGB9 pad 1: +5V -> C0_A
- RGB90 pad 1: +5V -> C0_A
- RGB91 pad 1: +5V -> C0_A
- RGB92 pad 1: +5V -> C0_A
- RGB93 pad 1: +5V -> C0_A
- RGB94 pad 1: +5V -> C0_A
- RGB95 pad 1: +5V -> C0_A
- RGB96 pad 1: +5V -> C0_A
- RGB97 pad 1: +5V -> C0_A
- RGB98 pad 1: +5V -> C0_A
- RGB99 pad 1: +5V -> C0_A
- SW10 pad 1: Net-(SW10-Pad1) -> Net-(R71-Pad2)
- SW100 pad 1: Net-(SW100-Pad1) -> SW6_2
- SW101 pad 1: Net-(SW101-Pad1) -> SW6_2
- SW102 pad 1: Net-(SW102-Pad1) -> SW6_2
- SW103 pad 1: Net-(SW103-Pad1) -> SW6_2
- SW104 pad 1: Net-(SW104-Pad1) -> SW7_2
- SW105 pad 1: Net-(SW105-Pad1) -> SW7_2
- SW106 pad 1: Net-(SW106-Pad1) -> SW7_2
- SW107 pad 1: Net-(SW107-Pad1) -> SW7_2
- SW108 pad 1: Net-(SW108-Pad1) -> SW7_2
- SW11 pad 1: Net-(SW11-Pad1) -> Net-(R71-Pad2)
- SW12 pad 1: Net-(SW12-Pad1) -> Net-(R71-Pad2)
- SW13 pad 1: Net-(SW13-Pad1) -> Net-(R72-Pad2)
- SW14 pad 1: Net-(SW14-Pad1) -> Net-(R72-Pad2)
- SW15 pad 1: Net-(SW15-Pad1) -> Net-(R72-Pad2)
- SW16 pad 1: Net-(SW16-Pad1) -> Net-(R72-Pad2)
- SW17 pad 1: Net-(SW17-Pad1) -> Net-(R72-Pad2)
- SW18 pad 1: Net-(SW18-Pad1) -> Net-(R72-Pad2)
- SW19 pad 1: Net-(SW19-Pad1) -> Net-(R73-Pad2)
- SW20 pad 1: Net-(SW20-Pad1) -> Net-(R73-Pad2)
- SW21 pad 1: Net-(SW21-Pad1) -> Net-(R73-Pad2)
- SW22 pad 1: Net-(SW22-Pad1) -> Net-(R73-Pad2)
- SW23 pad 1: Net-(SW23-Pad1) -> Net-(R73-Pad2)
- SW24 pad 1: Net-(SW24-Pad1) -> Net-(R73-Pad2)
- SW25 pad 1: Net-(SW25-Pad1) -> Net-(R74-Pad2)
- SW26 pad 1: Net-(SW26-Pad1) -> Net-(R74-Pad2)
- SW27 pad 1: Net-(SW27-Pad1) -> Net-(R74-Pad2)
- SW28 pad 1: Net-(SW28-Pad1) -> Net-(R74-Pad2)
- SW29 pad 1: Net-(SW29-Pad1) -> Net-(R74-Pad2)
- SW30 pad 1: Net-(SW30-Pad1) -> Net-(R75-Pad2)
- SW31 pad 1: Net-(SW31-Pad1) -> Net-(R75-Pad2)
- SW32 pad 1: Net-(SW32-Pad1) -> Net-(R75-Pad2)
- SW33 pad 1: Net-(SW33-Pad1) -> Net-(R75-Pad2)
- SW34 pad 1: Net-(SW34-Pad1) -> Net-(R76-Pad2)
- SW35 pad 1: Net-(SW35-Pad1) -> Net-(R76-Pad2)
- SW37 pad 1: Net-(SW37-Pad1) -> Net-(R78-Pad2)
- SW38 pad 1: Net-(SW38-Pad1) -> Net-(R78-Pad2)
- SW39 pad 1: Net-(SW39-Pad1) -> Net-(R78-Pad2)
- SW40 pad 1: Net-(SW40-Pad1) -> Net-(R78-Pad2)
- SW41 pad 1: Net-(SW41-Pad1) -> Net-(R79-Pad2)
- SW42 pad 1: Net-(SW42-Pad1) -> Net-(R79-Pad2)
- SW43 pad 1: Net-(SW43-Pad1) -> Net-(R79-Pad2)
- SW44 pad 1: Net-(SW44-Pad1) -> Net-(R79-Pad2)
- SW45 pad 1: Net-(SW45-Pad1) -> Net-(R79-Pad2)
- SW46 pad 1: Net-(SW46-Pad1) -> Net-(R80-Pad2)
- SW47 pad 1: Net-(SW47-Pad1) -> Net-(R80-Pad2)
- SW48 pad 1: Net-(SW48-Pad1) -> Net-(R80-Pad2)
- SW49 pad 1: Net-(SW49-Pad1) -> Net-(R80-Pad2)
- SW5 pad 1: Net-(SW5-Pad1) -> Net-(R70-Pad2)
- SW50 pad 1: Net-(SW50-Pad1) -> Net-(R80-Pad2)
- SW51 pad 1: Net-(SW51-Pad1) -> Net-(R80-Pad2)
- SW52 pad 1: Net-(SW52-Pad1) -> Net-(R81-Pad2)
- SW53 pad 1: Net-(SW53-Pad1) -> Net-(R81-Pad2)
- SW54 pad 1: Net-(SW54-Pad1) -> Net-(R81-Pad2)
- SW55 pad 1: Net-(SW55-Pad1) -> Net-(R81-Pad2)
- SW56 pad 1: Net-(SW56-Pad1) -> Net-(R81-Pad2)
- SW57 pad 1: Net-(SW57-Pad1) -> Net-(R81-Pad2)
- SW58 pad 1: Net-(SW58-Pad1) -> Net-(R82-Pad2)
- SW59 pad 1: Net-(SW59-Pad1) -> Net-(R82-Pad2)
- SW6 pad 1: Net-(SW6-Pad1) -> Net-(R70-Pad2)
- SW60 pad 1: Net-(SW60-Pad1) -> Net-(R82-Pad2)
- SW61 pad 1: Net-(SW61-Pad1) -> Net-(R82-Pad2)
- SW62 pad 1: Net-(SW62-Pad1) -> Net-(R82-Pad2)
- SW63 pad 1: Net-(SW63-Pad1) -> Net-(R82-Pad2)
- SW64 pad 1: Net-(SW64-Pad1) -> Net-(R83-Pad2)
- SW65 pad 1: Net-(SW65-Pad1) -> Net-(R83-Pad2)
- SW66 pad 1: Net-(SW66-Pad1) -> Net-(R83-Pad2)
- SW67 pad 1: Net-(SW67-Pad1) -> Net-(R83-Pad2)
- SW68 pad 1: Net-(SW68-Pad1) -> Net-(R83-Pad2)
- SW69 pad 1: Net-(SW69-Pad1) -> Net-(R83-Pad2)
- SW7 pad 1: Net-(SW7-Pad1) -> Net-(R71-Pad2)
- SW70 pad 1: Net-(SW70-Pad1) -> Net-(R84-Pad2)
- SW71 pad 1: Net-(SW71-Pad1) -> Net-(R84-Pad2)
- SW72 pad 1: Net-(SW72-Pad1) -> Net-(R84-Pad2)
- SW73 pad 1: Net-(SW73-Pad1) -> Net-(R84-Pad2)
- SW74 pad 1: Net-(SW74-Pad1) -> Net-(R84-Pad2)
- SW75 pad 1: Net-(SW75-Pad1) -> Net-(R84-Pad2)
- SW76 pad 1: Net-(SW76-Pad1) -> Net-(R85-Pad2)
- SW77 pad 1: Net-(SW77-Pad1) -> Net-(R85-Pad2)
- SW78 pad 1: Net-(SW78-Pad1) -> Net-(R85-Pad2)
- SW79 pad 1: Net-(SW79-Pad1) -> Net-(R85-Pad2)
- SW8 pad 1: Net-(SW8-Pad1) -> Net-(R71-Pad2)
- SW80 pad 1: Net-(SW80-Pad1) -> Net-(R86-Pad2)
- SW81 pad 1: Net-(SW81-Pad1) -> Net-(R86-Pad2)
- SW82 pad 1: Net-(SW82-Pad1) -> Net-(R86-Pad2)
- SW83 pad 1: Net-(SW83-Pad1) -> Net-(R86-Pad2)
- SW84 pad 1: Net-(SW84-Pad1) -> Net-(R86-Pad2)
- SW85 pad 1: Net-(SW85-Pad1) -> Net-(R87-Pad2)
- SW86 pad 1: Net-(SW86-Pad1) -> Net-(R87-Pad2)
- SW87 pad 1: Net-(SW87-Pad1) -> Net-(R87-Pad2)
- SW88 pad 1: Net-(SW88-Pad1) -> Net-(R87-Pad2)
- SW89 pad 1: Net-(SW89-Pad1) -> SW4_2
- SW9 pad 1: Net-(SW9-Pad1) -> Net-(R71-Pad2)
- SW90 pad 1: Net-(SW90-Pad1) -> SW4_2
- SW91 pad 1: Net-(SW91-Pad1) -> SW4_2
- SW92 pad 1: Net-(SW92-Pad1) -> SW4_2
- SW93 pad 1: Net-(SW93-Pad1) -> SW4_2
- SW94 pad 1: Net-(SW94-Pad1) -> SW5_2
- SW95 pad 1: Net-(SW95-Pad1) -> SW5_2
- SW96 pad 1: Net-(SW96-Pad1) -> SW5_2
- SW97 pad 1: Net-(SW97-Pad1) -> SW5_2
- SW98 pad 1: Net-(SW98-Pad1) -> SW5_2
- SW99 pad 1: Net-(SW99-Pad1) -> SW6_2
- U1 pad 1: D7 -> Net-(U1-Pad1)
- U1 pad 10: MOSI -> Net-(U1-Pad1)
- U1 pad 11: MISO -> D-_A
- U1 pad 12: D11 -> D+_A
- U1 pad 13: Net-(R25-Pad2) -> Net-(R37-Pad1)
- U1 pad 14: +5V -> GND
- U1 pad 16: Net-(C3-Pad1) -> Net-(U1-Pad1)
- U1 pad 17: Net-(C2-Pad1) -> GND
- U1 pad 18: D3 -> GND
- U1 pad 19: D2 -> unconnected-(U1-Pad19)
- U1 pad 2: +5V -> unconnected-(U1-Pad2)
- U1 pad 20: D0 -> unconnected-(U1-Pad20)
- U1 pad 21: D1 -> unconnected-(U1-Pad21)
- U1 pad 22: Net-(R28-Pad1) -> unconnected-(U1-Pad22)
- U1 pad 23: GND -> C0_A
- U1 pad 24: +5V -> Net-(U1-Pad1)
- U1 pad 25: D4 -> Net-(U1-Pad25)
- U1 pad 26: D12 -> Net-(U1-Pad26)
- U1 pad 27: D6 -> Net-(U1-Pad27)
- U1 pad 28: D8 -> Net-(U1-Pad28)
- U1 pad 3: Net-(R27-Pad2) -> unconnected-(U1-Pad3)
- U1 pad 4: Net-(R26-Pad1) -> Net-(R36-Pad1)
- U1 pad 5: GND -> Net-(U1-Pad1)
- U1 pad 6: Net-(C5-Pad1) -> Net-(C7-Pad1)
- U1 pad 7: +5V -> Net-(C6-Pad1)
- U1 pad 8: D14 -> unconnected-(U1-Pad8)
- U1 pad 9: SCK -> unconnected-(U1-Pad9)
- U2 pad 1: D7 -> Net-(U2-Pad1)
- U2 pad 10: MOSI -> Net-(U2-Pad1)
- U2 pad 11: MISO -> L_D-
- U2 pad 12: D11 -> L_D+
- U2 pad 13: Net-(R32-Pad2) -> Net-(R39-Pad1)
- U2 pad 14: +5V -> GND
- U2 pad 16: Net-(C9-Pad1) -> Net-(U2-Pad1)
- U2 pad 17: Net-(C8-Pad1) -> GND
- U2 pad 18: D3 -> GND
- U2 pad 19: D2 -> unconnected-(U2-Pad19)
- U2 pad 2: +5V -> LEFT3 D-
- U2 pad 20: D0 -> unconnected-(U2-Pad20)
- U2 pad 21: D1 -> unconnected-(U2-Pad21)
- U2 pad 22: Net-(R42-Pad1) -> unconnected-(U2-Pad22)
- U2 pad 23: GND -> C0_A
- U2 pad 24: +5V -> Net-(U2-Pad1)
- U2 pad 25: D4 -> LEFT1 D-
- U2 pad 26: D12 -> LEFT1 D+
- U2 pad 27: D6 -> LEFT2 D-
- U2 pad 28: D8 -> LEFT2 D+
- U2 pad 3: Net-(R40-Pad2) -> LEFT3 D+
- U2 pad 5: GND -> Net-(U2-Pad1)
- U2 pad 6: Net-(C14-Pad1) -> Net-(C9-Pad1)
- U2 pad 7: +5V -> Net-(C8-Pad1)
- U2 pad 8: D14 -> LEFT4 D-
- U2 pad 9: SCK -> LEFT4 D+
- U3 pad 1: D7 -> Net-(U3-Pad1)
- U3 pad 10: MOSI -> Net-(U3-Pad1)
- U3 pad 11: MISO -> D-_N
- U3 pad 12: D11 -> D+_N
- U3 pad 13: Net-(R33-Pad2) -> Net-(R49-Pad1)
- U3 pad 14: +5V -> GND
- U3 pad 16: Net-(C11-Pad1) -> Net-(U3-Pad1)
- U3 pad 17: Net-(C10-Pad1) -> GND
- U3 pad 18: D3 -> GND
- U3 pad 19: D2 -> unconnected-(U3-Pad19)
- U3 pad 2: +5V -> unconnected-(U3-Pad2)
- U3 pad 20: D0 -> unconnected-(U3-Pad20)
- U3 pad 21: D1 -> unconnected-(U3-Pad21)
- U3 pad 22: Net-(R44-Pad1) -> unconnected-(U3-Pad22)
- U3 pad 23: GND -> C0_A
- U3 pad 24: +5V -> Net-(U3-Pad1)
- U3 pad 25: D4 -> Net-(U3-Pad25)
- U3 pad 26: D12 -> Net-(U3-Pad26)
- U3 pad 27: D6 -> Net-(U3-Pad27)
- U3 pad 28: D8 -> Net-(U3-Pad28)
- U3 pad 3: Net-(R41-Pad2) -> unconnected-(U3-Pad3)
- U3 pad 4: Net-(R39-Pad1) -> Net-(R48-Pad1)
- U3 pad 5: GND -> Net-(U3-Pad1)
- U3 pad 6: Net-(C15-Pad1) -> Net-(C11-Pad1)
- U3 pad 7: +5V -> Net-(C10-Pad1)
- U3 pad 8: D14 -> unconnected-(U3-Pad8)
- U3 pad 9: SCK -> unconnected-(U3-Pad9)
- USB1 pad A4: +5V -> C0_A
- USB1 pad A5: Net-(R2-Pad2) -> Net-(R30-Pad1)
- USB1 pad A6: D+ -> Net-(U1-Pad26)
- USB1 pad A7: D- -> Net-(U1-Pad25)
- USB1 pad A8: Net-(USB1-PadA8) -> unconnected-(USB1-PadA8)
- USB1 pad A9: +5V -> C0_A
- USB1 pad B4: +5V -> C0_A
- USB1 pad B5: Net-(R3-Pad1) -> Net-(R31-Pad1)
- USB1 pad B6: D+ -> Net-(U1-Pad26)
- USB1 pad B7: D- -> Net-(U1-Pad25)
- USB1 pad B8: Net-(USB1-PadB8) -> unconnected-(USB1-PadB8)
- USB1 pad B9: +5V -> C0_A
- USB3 pad A1: Net-(USB3-PadA1) -> GND
- USB3 pad A12: Net-(USB3-PadA1) -> GND
- USB3 pad A4: Net-(USB3-PadA4) -> C0_A
- USB3 pad A5: Net-(USB3-PadA5) -> Net-(R34-Pad1)
- USB3 pad A6: Net-(USB3-PadA6) -> LEFT1 D+
- USB3 pad A7: Net-(USB3-PadA7) -> LEFT1 D-
- USB3 pad A8: Net-(USB3-PadA8) -> RGB_IN_L
- USB3 pad A9: Net-(USB3-PadA4) -> C0_A
- USB3 pad B1: Net-(USB3-PadA1) -> GND
- USB3 pad B12: Net-(USB3-PadA1) -> GND
- USB3 pad B4: Net-(USB3-PadA4) -> C0_A
- USB3 pad B5: Net-(USB3-PadB5) -> Net-(R35-Pad1)
- USB3 pad B6: Net-(USB3-PadB6) -> LEFT1 D+
- USB3 pad B7: Net-(USB3-PadB7) -> LEFT1 D-
- USB3 pad B8: Net-(USB3-PadB8) -> RGB_IN_L
- USB3 pad B9: Net-(USB3-PadA4) -> C0_A
- USB3 pad S1: Net-(USB3-PadS1) -> GND
- USB4 pad A4: +5V -> C0_A
- USB4 pad A5: Net-(R34-Pad2) -> Net-(R32-Pad1)
- USB4 pad A6: Net-(R40-Pad1) -> LEFT2 D+
- USB4 pad A7: Net-(R38-Pad2) -> LEFT2 D-
- USB4 pad A8: Net-(USB4-PadA8) -> RGB_OUT_L
- USB4 pad A9: +5V -> C0_A
- USB4 pad B4: +5V -> C0_A
- USB4 pad B5: Net-(R36-Pad1) -> Net-(R33-Pad1)
- USB4 pad B6: Net-(R40-Pad1) -> LEFT2 D+
- USB4 pad B7: Net-(R38-Pad2) -> LEFT2 D-
- USB4 pad B8: Net-(USB4-PadB8) -> RGB_OUT_L
- USB4 pad B9: +5V -> C0_A
- USB7 pad A1: Net-(USB7-PadA1) -> GND
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Routing:
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Other:
- outline, holes or cut-outs redrawn
- net class Default removed
